File: USBTINYISP_MICRO_USB.sch (KiCad schematic (older format))
At the start: 17 parts, among them J1 USB_B_Micro, J2 AVR-ISP-6, U1 ATtiny84-20PU, Y1 12MHZ

Commit message: update
Parts:
- removed JP1: Jumper_NC_Small, symbol Device:Jumper_NC_Small
- added D?: LED_data+, symbol Device:LED_Small_ALT
- added D?: LED_data-, symbol Device:LED_Small_ALT
- added D?: LED_SCK, symbol Device:LED_Small_ALT
- added D?: LED_power, symbol Device:LED_Small_ALT
- added JP1: Rest_connect, Jumper:SolderJumper-2_P1.3mm_Open_TrianglePad1.0x1.5mm, symbol Device:Jumper_NO_Small
- added R? (x4): 1k, Resistor_THT:R_Axial_DIN0204_L3.6mm_D1.6mm_P1.90mm_Vertical, symbol Device:R_US
- C1, C2, C3, C4: footprint (none) -> Capacitor_THT:C_Disc_D3.0mm_W1.6mm_P2.50mm
- D1, D2: footprint (none) -> Diode_THT:D_DO-15_P2.54mm_Vertical_AnodeUp
- J1: footprint (none) -> Connector_USB:USB_Micro-B_Molex_47346-0001
- J2: footprint (none) -> Connector_PinHeader_2.54mm:PinHeader_2x03_P2.54mm_Vertical
- JP2: value Jumper_NC_Small -> USB_power; footprint (none) -> Jumper:SolderJumper-2_P1.3mm_Bridged2Bar_RoundedPad1.0x1.5mm
- R1, R2, R3, R4, R5: footprint (none) -> Resistor_THT:R_Axial_DIN0204_L3.6mm_D1.6mm_P1.90mm_Vertical
- Y1: footprint (none) -> Crystal:Crystal_HC49-4H_Vertical
Connections:
- net D+: now also R?.1
- net D-: now also R?.1
- net GND: now also D?.1 (K), D?.1 (K), D?.1 (K), D?.1 (K)
- net SCK: now also R?.1
- net VCC: now also R?.1
- net at R2.1, U1.4 (~RESET~/PB3): now also JP1.2
- net at R1.1: now also JP1.1
- new net: D?.2 (A), R?.2 (x4)
- no-connect marks 3 -> 4
Other:
- note added: "LED to know the status"
- moved on the sheet: C1, C2, R1, R2, U1, Y1

Commit message: update
Parts:
- D1, D4: renamed from D?; footprint (none) -> LED_THT:LED_D3.0mm
- D2, D3: renamed from D?; footprint (none) -> LED_THT:LED_D3.0mm_Clear
- gave numbers to parts that had none: 4
- renumbered D1 to D5, D2 to D6, R1 to R4, R2 to R5, R3 to R7, R4 to R8, R5 to R9
Changed lines of the file:
@@
 $EndComp
 $Comp
-L power:GND #PWR03
+L power:GND #PWR04
 U 1 1 5EF8E156
 P 6650 6190
-F 0 "#PWR03" H 6650 5940 50  0001 C CNN
+F 0 "#PWR04" H 6650 5940 50  0001 C CNN
 F 1 "GND" H 6655 6017 50  0000 C CNN
 F 2 "" H 6650 6190 50  0001 C CNN
@@
 $EndComp
 $Comp
-L Device:R_US R2
+L Device:R_US R5
 U 1 1 5EF8EE28
 P 3590 3280
-F 0 "R2" H 3658 3326 50  0000 L CNN
+F 0 "R5" H 3658 3326 50  0000 L CNN
 F 1 "10k" H 3658 3235 50  0000 L CNN
 F 2 "Resistor_THT:R_Axial_DIN0204_L3.6mm_D1.6mm_P1.90mm_Vertical" V 3630 3270 50  0001 C CNN
@@
 	7010 5490 7290 5490
 $Comp
-L Device:D_Zener_Small D2
+L Device:D_Zener_Small D6
 U 1 1 5EF9208F
 P 7950 5790
-F 0 "D2" V 7904 5860 50  0000 L CNN
+F 0 "D6" V 7904 5860 50  0000 L CNN
 F 1 "3v3" V 7995 5860 50  0000 L CNN
 F 2 "Diode_THT:D_DO-15_P2.54mm_Vertical_AnodeUp" V 7950 5790 50  0001 C CNN
@@
 $EndComp
 $Comp
-L Device:R_US R4
+L Device:R_US R8
 U 1 1 5EF92A54
 P 7680 5790
-F 0 "R4" V 7475 5790 50  0000 C CNN
+F 0 "R8" V 7475 5790 50  0000 C CNN
 F 1 "68" V 7566 5790 50  0000 C CNN
 F 2 "Resistor_THT:R_Axial_DIN0204_L3.6mm_D1.6mm_P1.90mm_Vertical" V 7720 5780 50  0001 C CNN
@@
 $EndComp
 $Comp
-L Device:R_US R5
+L Device:R_US R9
 U 1 1 5EF9363C
 P 8170 5690
-F 0 "R5" V 7965 5690 50  0000 C CNN
+F 0 "R9" V 7965 5690 50  0000 C CNN
 F 1 "68" V 8056 5690 50  0000 C CNN
 F 2 "Resistor_THT:R_Axial_DIN0204_L3.6mm_D1.6mm_P1.90mm_Vertical" V 8210 5680 50  0001 C CNN
@@
 	7830 5790 8580 5790
 $Comp
-L Device:D_Zener_Small D1
+L Device:D_Zener_Small D5
 U 1 1 5EF95067
 P 7290 5890
-F 0 "D1" V 7244 5960 50  0000 L CNN
+F 0 "D5" V 7244 5960 50  0000 L CNN
 F 1 "3v3" V 7335 5960 50  0000 L CNN
 F 2 "Diode_THT:D_DO-15_P2.54mm_Vertical_AnodeUp" V 7290 5890 50  0001 C CNN
@@
 	7950 5690 8020 5690
 $Comp
-L power:GND #PWR04
+L power:GND #PWR05
 U 1 1 5EF960C8
 P 7290 5990
-F 0 "#PWR04" H 7290 5740 50  0001 C CNN
+F 0 "#PWR05" H 7290 5740 50  0001 C CNN
 F 1 "GND" H 7295 5817 50  0000 C CNN
 F 2 "" H 7290 5990 50  0001 C CNN
@@
 $EndComp
 $Comp
-L power:GND #PWR07
+L power:GND #PWR08
 U 1 1 5EF9677B
 P 7950 5890
-F 0 "#PWR07" H 7950 5640 50  0001 C CNN
+F 0 "#PWR08" H 7950 5640 50  0001 C CNN
 F 1 "GND" H 7955 5717 50  0000 C CNN
 F 2 "" H 7950 5890 50  0001 C CNN
@@
 $EndComp
 $Comp
-L Device:R_US R3
+L Device:R_US R7
 U 1 1 5EF96EA8
 P 7290 5640
-F 0 "R3" H 7358 5686 50  0000 L CNN
+F 0 "R7" H 7358 5686 50  0000 L CNN
 F 1 "1.5k" H 7358 5595 50  0000 L CNN
 F 2 "Resistor_THT:R_Axial_DIN0204_L3.6mm_D1.6mm_P1.90mm_Vertical" V 7330 5630 50  0001 C CNN
@@
 $EndComp
 $Comp
-L power:GND #PWR06
+L power:GND #PWR07
 U 1 1 5EF9ED1A
 P 7740 1690
-F 0 "#PWR06" H 7740 1440 50  0001 C CNN
+F 0 "#PWR07" H 7740 1440 50  0001 C CNN
 F 1 "GND" H 7745 1517 50  0000 C CNN
 F 2 "" H 7740 1690 50  0001 C CNN
@@
 $EndComp
 $Comp
-L power:GND #PWR05
+L power:GND #PWR06
 U 1 1 5EF9F648
 P 7310 3860
-F 0 "#PWR05" H 7310 3610 50  0001 C CNN
+F 0 "#PWR06" H 7310 3610 50  0001 C CNN
 F 1 "GND" H 7315 3687 50  0000 C CNN
 F 2 "" H 7310 3860 50  0001 C CNN
@@
 	3920 2630 3920 2740
 $Comp
-L power:GND #PWR02
+L power:GND #PWR03
 U 1 1 5EFA76FA
 P 4000 2630
-F 0 "#PWR02" H 4000 2380 50  0001 C CNN
+F 0 "#PWR03" H 4000 2380 50  0001 C CNN
 F 1 "GND" V 4005 2502 50  0000 R CNN
 F 2 "" H 4000 2630 50  0001 C CNN
@@
 	3450 3330 3450 3540
 $Comp
-L Device:R_US R1
+L Device:R_US R4
 U 1 1 5EFBE903
 P 3450 3690
-F 0 "R1" H 3518 3736 50  0000 L CNN
+F 0 "R4" H 3518 3736 50  0000 L CNN
 F 1 "0" H 3518 3645 50  0000 L CNN
 F 2 "Resistor_THT:R_Axial_DIN0204_L3.6mm_D1.6mm_P1.90mm_Vertical" V 3490 3680 50  0001 C CNN
@@
 LED to know the status
 $Comp
-L Device:LED_Small_ALT D?
+L Device:LED_Small_ALT D2
 U 1 1 5EFD7759
 P 2490 7080
-F 0 "D?" V 2536 7010 50  0000 R CNN
+F 0 "D2" V 2536 7010 50  0000 R CNN
 F 1 "LED_data+" V 2445 7010 50  0000 R CNN
-F 2 "" V 2490 7080 50  0001 C CNN
+F 2 "LED_THT:LED_D3.0mm_Clear" V 2490 7080 50  0001 C CNN
 F 3 "~" V 2490 7080 50  0001 C CNN
 	1    2490 7080
@@
 $EndComp
 $Comp
-L Device:LED_Small_ALT D?
+L Device:LED_Small_ALT D3
 U 1 1 5EFD84EB
 P 3330 7080
-F 0 "D?" V 3376 7010 50  0000 R CNN
+F 0 "D3" V 3376 7010 50  0000 R CNN
 F 1 "LED_data-" V 3285 7010 50  0000 R CNN
-F 2 "" V 3330 7080 50  0001 C CNN
+F 2 "LED_THT:LED_D3.0mm_Clear" V 3330 7080 50  0001 C CNN
 F 3 "~" V 3330 7080 50  0001 C CNN
 	1    3330 7080
@@
 $EndComp
 $Comp
-L Device:LED_Small_ALT D?
+L Device:LED_Small_ALT D4
 U 1 1 5EFD88A0
 P 4370 7080
-F 0 "D?" V 4416 7010 50  0000 R CNN
+F 0 "D4" V 4416 7010 50  0000 R CNN
 F 1 "LED_SCK" V 4325 7010 50  0000 R CNN
-F 2 "" V 4370 7080 50  0001 C CNN
+F 2 "LED_THT:LED_D3.0mm" V 4370 7080 50  0001 C CNN
 F 3 "~" V 4370 7080 50  0001 C CNN
 	1    4370 7080
@@
 $EndComp
 $Comp
-L Device:R_US R?
+L Device:R_US R2
 U 1 1 5EFD8DF9
 P 2490 6830
-F 0 "R?" H 2558 6876 50  0000 L CNN
+F 0 "R2" H 2558 6876 50  0000 L CNN
 F 1 "1k" H 2558 6785 50  0000 L CNN
 F 2 "Resistor_THT:R_Axial_DIN0204_L3.6mm_D1.6mm_P1.90mm_Vertical" V 2530 6820 50  0001 C CNN
@@
 $EndComp
 $Comp
-L Device:R_US R?
+L Device:R_US R3
 U 1 1 5EFD9C83
 P 3330 6830
-F 0 "R?" H 3398 6876 50  0000 L CNN
+F 0 "R3" H 3398 6876 50  0000 L CNN
 F 1 "1k" H 3398 6785 50  0000 L CNN
 F 2 "Resistor_THT:R_Axial_DIN0204_L3.6mm_D1.6mm_P1.90mm_Vertical" V 3370 6820 50  0001 C CNN
@@
 $EndComp
 $Comp
-L Device:R_US R?
+L Device:R_US R6
 U 1 1 5EFDA4D7
 P 4370 6830
-F 0 "R?" H 4438 6876 50  0000 L CNN
+F 0 "R6" H 4438 6876 50  0000 L CNN
 F 1 "1k" H 4438 6785 50  0000 L CNN
 F 2 "Resistor_THT:R_Axial_DIN0204_L3.6mm_D1.6mm_P1.90mm_Vertical" V 4410 6820 50  0001 C CNN
@@
 	3330 7180 4370 7180
 $Comp
-L power:GND #PWR?
+L power:GND #PWR02
 U 1 1 5EFE066D
 P 3330 7180
-F 0 "#PWR?" H 3330 6930 50  0001 C CNN
+F 0 "#PWR02" H 3330 6930 50  0001 C CNN
 F 1 "GND" H 3335 7007 50  0000 C CNN
 F 2 "" H 3330 7180 50  0001 C CNN
@@
 SCK
 $Comp
-L Device:LED_Small_ALT D?
+L Device:LED_Small_ALT D1
 U 1 1 5EFE74E4
 P 1770 7080
-F 0 "D?" V 1816 7010 50  0000 R CNN
+F 0 "D1" V 1816 7010 50  0000 R CNN
 F 1 "LED_power" V 1725 7010 50  0000 R CNN
-F 2 "" V 1770 7080 50  0001 C CNN
+F 2 "LED_THT:LED_D3.0mm" V 1770 7080 50  0001 C CNN
 F 3 "~" V 1770 7080 50  0001 C CNN
 	1    1770 7080
@@
 $EndComp
 $Comp
-L Device:R_US R?
+L Device:R_US R1
 U 1 1 5EFE74EA
 P 1770 6830
-F 0 "R?" H 1838 6876 50  0000 L CNN
+F 0 "R1" H 1838 6876 50  0000 L CNN
 F 1 "1k" H 1838 6785 50  0000 L CNN
 F 2 "Resistor_THT:R_Axial_DIN0204_L3.6mm_D1.6mm_P1.90mm_Vertical" V 1810 6820 50  0001 C CNN

Commit message: update
Parts:
- D5, D6: footprint Diode_THT:D_DO-15_P2.54mm_Vertical_AnodeUp -> Diode_THT:D_DO-41_SOD81_P2.54mm_Vertical_AnodeUp
- R1, R2, R3, R4, R5, R6, R7, R8, R9: footprint Resistor_THT:R_Axial_DIN0204_L3.6mm_D1.6mm_P1.90mm_Vertical -> Resistor_THT:R_Axial_DIN0207_L6.3mm_D2.5mm_P2.54mm_Vertical
Changed lines of the file:
@@
 F 0 "R5" H 3658 3326 50  0000 L CNN
 F 1 "10k" H 3658 3235 50  0000 L CNN
-F 2 "Resistor_THT:R_Axial_DIN0204_L3.6mm_D1.6mm_P1.90mm_Vertical" V 3630 3270 50  0001 C CNN
+F 2 "Resistor_THT:R_Axial_DIN0207_L6.3mm_D2.5mm_P2.54mm_Vertical" V 3630 3270 50  0001 C CNN
 F 3 "~" H 3590 3280 50  0001 C CNN
 	1    3590 3280
@@
 F 0 "D6" V 7904 5860 50  0000 L CNN
 F 1 "3v3" V 7995 5860 50  0000 L CNN
-F 2 "Diode_THT:D_DO-15_P2.54mm_Vertical_AnodeUp" V 7950 5790 50  0001 C CNN
+F 2 "Diode_THT:D_DO-41_SOD81_P2.54mm_Vertical_AnodeUp" V 7950 5790 50  0001 C CNN
 F 3 "~" V 7950 5790 50  0001 C CNN
 	1    7950 5790
@@
 F 0 "R8" V 7475 5790 50  0000 C CNN
 F 1 "68" V 7566 5790 50  0000 C CNN
-F 2 "Resistor_THT:R_Axial_DIN0204_L3.6mm_D1.6mm_P1.90mm_Vertical" V 7720 5780 50  0001 C CNN
+F 2 "Resistor_THT:R_Axial_DIN0207_L6.3mm_D2.5mm_P2.54mm_Vertical" V 7720 5780 50  0001 C CNN
 F 3 "~" H 7680 5790 50  0001 C CNN
 	1    7680 5790
@@
 F 0 "R9" V 7965 5690 50  0000 C CNN
 F 1 "68" V 8056 5690 50  0000 C CNN
-F 2 "Resistor_THT:R_Axial_DIN0204_L3.6mm_D1.6mm_P1.90mm_Vertical" V 8210 5680 50  0001 C CNN
+F 2 "Resistor_THT:R_Axial_DIN0207_L6.3mm_D2.5mm_P2.54mm_Vertical" V 8210 5680 50  0001 C CNN
 F 3 "~" H 8170 5690 50  0001 C CNN
 	1    8170 5690
@@
 F 0 "D5" V 7244 5960 50  0000 L CNN
 F 1 "3v3" V 7335 5960 50  0000 L CNN
-F 2 "Diode_THT:D_DO-15_P2.54mm_Vertical_AnodeUp" V 7290 5890 50  0001 C CNN
+F 2 "Diode_THT:D_DO-41_SOD81_P2.54mm_Vertical_AnodeUp" V 7290 5890 50  0001 C CNN
 F 3 "~" V 7290 5890 50  0001 C CNN
 	1    7290 5890
@@
 F 0 "R7" H 7358 5686 50  0000 L CNN
 F 1 "1.5k" H 7358 5595 50  0000 L CNN
-F 2 "Resistor_THT:R_Axial_DIN0204_L3.6mm_D1.6mm_P1.90mm_Vertical" V 7330 5630 50  0001 C CNN
+F 2 "Resistor_THT:R_Axial_DIN0207_L6.3mm_D2.5mm_P2.54mm_Vertical" V 7330 5630 50  0001 C CNN
 F 3 "~" H 7290 5640 50  0001 C CNN
 	1    7290 5640
@@
 F 0 "R4" H 3518 3736 50  0000 L CNN
 F 1 "0" H 3518 3645 50  0000 L CNN
-F 2 "Resistor_THT:R_Axial_DIN0204_L3.6mm_D1.6mm_P1.90mm_Vertical" V 3490 3680 50  0001 C CNN
+F 2 "Resistor_THT:R_Axial_DIN0207_L6.3mm_D2.5mm_P2.54mm_Vertical" V 3490 3680 50  0001 C CNN
 F 3 "~" H 3450 3690 50  0001 C CNN
 	1    3450 3690
@@
 F 0 "R2" H 2558 6876 50  0000 L CNN
 F 1 "1k" H 2558 6785 50  0000 L CNN
-F 2 "Resistor_THT:R_Axial_DIN0204_L3.6mm_D1.6mm_P1.90mm_Vertical" V 2530 6820 50  0001 C CNN
+F 2 "Resistor_THT:R_Axial_DIN0207_L6.3mm_D2.5mm_P2.54mm_Vertical" V 2530 6820 50  0001 C CNN
 F 3 "~" H 2490 6830 50  0001 C CNN
 	1    2490 6830
@@
 F 0 "R3" H 3398 6876 50  0000 L CNN
 F 1 "1k" H 3398 6785 50  0000 L CNN
-F 2 "Resistor_THT:R_Axial_DIN0204_L3.6mm_D1.6mm_P1.90mm_Vertical" V 3370 6820 50  0001 C CNN
+F 2 "Resistor_THT:R_Axial_DIN0207_L6.3mm_D2.5mm_P2.54mm_Vertical" V 3370 6820 50  0001 C CNN
 F 3 "~" H 3330 6830 50  0001 C CNN
 	1    3330 6830
@@
 F 0 "R6" H 4438 6876 50  0000 L CNN
 F 1 "1k" H 4438 6785 50  0000 L CNN
-F 2 "Resistor_THT:R_Axial_DIN0204_L3.6mm_D1.6mm_P1.90mm_Vertical" V 4410 6820 50  0001 C CNN
+F 2 "Resistor_THT:R_Axial_DIN0207_L6.3mm_D2.5mm_P2.54mm_Vertical" V 4410 6820 50  0001 C CNN
 F 3 "~" H 4370 6830 50  0001 C CNN
 	1    4370 6830
@@
 F 0 "R1" H 1838 6876 50  0000 L CNN
 F 1 "1k" H 1838 6785 50  0000 L CNN
-F 2 "Resistor_THT:R_Axial_DIN0204_L3.6mm_D1.6mm_P1.90mm_Vertical" V 1810 6820 50  0001 C CNN
+F 2 "Resistor_THT:R_Axial_DIN0207_L6.3mm_D2.5mm_P2.54mm_Vertical" V 1810 6820 50  0001 C CNN
 F 3 "~" H 1770 6830 50  0001 C CNN
 	1    1770 6830

Commit message: update
Parts:
- removed D2: LED_data+, LED_THT:LED_D3.0mm_Clear, symbol Device:LED_Small_ALT
- removed D3: LED_data-, LED_THT:LED_D3.0mm_Clear, symbol Device:LED_Small_ALT
- removed R2, R3: 1k, Resistor_THT:R_Axial_DIN0207_L6.3mm_D2.5mm_P2.54mm_Vertical, symbol Device:R_US
- C1, C2, C3, C4: footprint Capacitor_THT:C_Disc_D3.0mm_W1.6mm_P2.50mm -> Capacitor_SMD:C_0805_2012Metric_Pad1.15x1.40mm_HandSolder
- D1, D4: footprint LED_THT:LED_D3.0mm -> LED_SMD:LED_0805_2012Metric_Pad1.15x1.40mm_HandSolder
- D5, D6: footprint Diode_THT:D_DO-41_SOD81_P2.54mm_Vertical_AnodeUp -> Diode_SMD:D_0805_2012Metric_Pad1.15x1.40mm_HandSolder
- J2: footprint Connector_PinHeader_2.54mm:PinHeader_2x03_P2.54mm_Vertical -> Connector_PinHeader_2.54mm:PinHeader_2x03_P2.54mm_Vertical_SMD
- JP1: footprint Jumper:SolderJumper-2_P1.3mm_Open_TrianglePad1.0x1.5mm -> Jumper:SolderJumper-2_P1.3mm_Open_RoundedPad1.0x1.5mm
- R1, R4, R5, R6, R7, R8, R9: footprint Resistor_THT:R_Axial_DIN0207_L6.3mm_D2.5mm_P2.54mm_Vertical -> Resistor_SMD:R_0805_2012Metric_Pad1.15x1.40mm_HandSolder
- U1: footprint Package_DIP:DIP-14_W7.62mm -> Package_SO:SOIC-14_3.9x8.7mm_P1.27mm; symbol MCU_Microchip_ATtiny:ATtiny84-20PU -> MCU_Microchip_ATtiny:ATtiny84A-SSU
- Y1: footprint Crystal:Crystal_HC49-4H_Vertical -> Crystal:Crystal_SMD_HC49-SD
Changed lines of the file:
@@
 F 0 "R5" H 3658 3326 50  0000 L CNN
 F 1 "10k" H 3658 3235 50  0000 L CNN
-F 2 "Resistor_THT:R_Axial_DIN0207_L6.3mm_D2.5mm_P2.54mm_Vertical" V 3630 3270 50  0001 C CNN
+F 2 "Resistor_SMD:R_0805_2012Metric_Pad1.15x1.40mm_HandSolder" V 3630 3270 50  0001 C CNN
 F 3 "~" H 3590 3280 50  0001 C CNN
 	1    3590 3280
@@
 F 0 "C1" V 3660 2530 50  0000 C CNN
 F 1 "18pf" V 3720 2550 50  0000 C CNN
-F 2 "Capacitor_THT:C_Disc_D3.0mm_W1.6mm_P2.50mm" H 3820 2540 50  0001 C CNN
+F 2 "Capacitor_SMD:C_0805_2012Metric_Pad1.15x1.40mm_HandSolder" H 3820 2540 50  0001 C CNN
 F 3 "~" H 3820 2540 50  0001 C CNN
 	1    3820 2540
@@
 F 0 "Y1" V 3720 2590 50  0000 L CNN
 F 1 "12MHZ" H 3460 2540 50  0000 L CNN
-F 2 "Crystal:Crystal_HC49-4H_Vertical" H 3720 2640 50  0001 C CNN
+F 2 "Crystal:Crystal_SMD_HC49-SD" H 3720 2640 50  0001 C CNN
 F 3 "~" H 3720 2640 50  0001 C CNN
 	1    3720 2640
@@
 F 0 "D6" V 7904 5860 50  0000 L CNN
 F 1 "3v3" V 7995 5860 50  0000 L CNN
-F 2 "Diode_THT:D_DO-41_SOD81_P2.54mm_Vertical_AnodeUp" V 7950 5790 50  0001 C CNN
+F 2 "Diode_SMD:D_0805_2012Metric_Pad1.15x1.40mm_HandSolder" V 7950 5790 50  0001 C CNN
 F 3 "~" V 7950 5790 50  0001 C CNN
 	1    7950 5790
@@
 F 0 "R8" V 7475 5790 50  0000 C CNN
 F 1 "68" V 7566 5790 50  0000 C CNN
-F 2 "Resistor_THT:R_Axial_DIN0207_L6.3mm_D2.5mm_P2.54mm_Vertical" V 7720 5780 50  0001 C CNN
+F 2 "Resistor_SMD:R_0805_2012Metric_Pad1.15x1.40mm_HandSolder" V 7720 5780 50  0001 C CNN
 F 3 "~" H 7680 5790 50  0001 C CNN
 	1    7680 5790
@@
 F 0 "R9" V 7965 5690 50  0000 C CNN
 F 1 "68" V 8056 5690 50  0000 C CNN
-F 2 "Resistor_THT:R_Axial_DIN0207_L6.3mm_D2.5mm_P2.54mm_Vertical" V 8210 5680 50  0001 C CNN
+F 2 "Resistor_SMD:R_0805_2012Metric_Pad1.15x1.40mm_HandSolder" V 8210 5680 50  0001 C CNN
 F 3 "~" H 8170 5690 50  0001 C CNN
 	1    8170 5690
@@
 F 0 "D5" V 7244 5960 50  0000 L CNN
 F 1 "3v3" V 7335 5960 50  0000 L CNN
-F 2 "Diode_THT:D_DO-41_SOD81_P2.54mm_Vertical_AnodeUp" V 7290 5890 50  0001 C CNN
+F 2 "Diode_SMD:D_0805_2012Metric_Pad1.15x1.40mm_HandSolder" V 7290 5890 50  0001 C CNN
 F 3 "~" V 7290 5890 50  0001 C CNN
 	1    7290 5890
@@
 F 0 "R7" H 7358 5686 50  0000 L CNN
 F 1 "1.5k" H 7358 5595 50  0000 L CNN
-F 2 "Resistor_THT:R_Axial_DIN0207_L6.3mm_D2.5mm_P2.54mm_Vertical" V 7330 5630 50  0001 C CNN
+F 2 "Resistor_SMD:R_0805_2012Metric_Pad1.15x1.40mm_HandSolder" V 7330 5630 50  0001 C CNN
 F 3 "~" H 7290 5640 50  0001 C CNN
 	1    7290 5640
@@
 	7290 5490 7500 5490
 $Comp
-L MCU_Microchip_ATtiny:ATtiny84-20PU U1
+L MCU_Microchip_ATtiny:ATtiny84A-SSU U1
 U 1 1 5EF9B48D
 P 2800 2280
 F 0 "U1" H 2271 2326 50  0000 R CNN
 F 1 "ATtiny84-20PU" H 2271 2235 50  0000 R CNN
-F 2 "Package_DIP:DIP-14_W7.62mm" H 2800 2280 50  0001 C CIN
+F 2 "Package_SO:SOIC-14_3.9x8.7mm_P1.27mm" H 2800 2280 50  0001 C CIN
 F 3 "http://ww1.microchip.com/downloads/en/DeviceDoc/doc8006.pdf" H 2800 2280 50  0001 C CNN
 	1    2800 2280
@@
 F 0 "J2" H 7081 3556 50  0000 R CNN
 F 1 "AVR-ISP-6" H 7081 3465 50  0000 R CNN
-F 2 "Connector_PinHeader_2.54mm:PinHeader_2x03_P2.54mm_Vertical" V 7160 3510 50  0001 C CNN
+F 2 "Connector_PinHeader_2.54mm:PinHeader_2x03_P2.54mm_Vertical_SMD" V 7160 3510 50  0001 C CNN
 F 3 " ~" H 6135 2910 50  0001 C CNN
 	1    7410 3460
@@
 F 0 "C3" H 7480 1580 50  0000 L CNN
 F 1 "0.1uf" H 7350 1470 50  0000 L CNN
-F 2 "Capacitor_THT:C_Disc_D3.0mm_W1.6mm_P2.50mm" H 7670 1530 50  0001 C CNN
+F 2 "Capacitor_SMD:C_0805_2012Metric_Pad1.15x1.40mm_HandSolder" H 7670 1530 50  0001 C CNN
 F 3 "~" H 7670 1530 50  0001 C CNN
 	1    7670 1530
@@
 F 0 "C4" H 7922 1576 50  0000 L CNN
 F 1 "10uf" H 7922 1485 50  0000 L CNN
-F 2 "Capacitor_THT:C_Disc_D3.0mm_W1.6mm_P2.50mm" H 7830 1530 50  0001 C CNN
+F 2 "Capacitor_SMD:C_0805_2012Metric_Pad1.15x1.40mm_HandSolder" H 7830 1530 50  0001 C CNN
 F 3 "~" H 7830 1530 50  0001 C CNN
 	1    7830 1530
@@
 F 0 "C2" V 3990 2740 50  0000 C CNN
 F 1 "18pf" V 3910 2770 50  0000 C CNN
-F 2 "Capacitor_THT:C_Disc_D3.0mm_W1.6mm_P2.50mm" H 3820 2740 50  0001 C CNN
+F 2 "Capacitor_SMD:C_0805_2012Metric_Pad1.15x1.40mm_HandSolder" H 3820 2740 50  0001 C CNN
 F 3 "~" H 3820 2740 50  0001 C CNN
 	1    3820 2740
@@
 F 0 "R4" H 3518 3736 50  0000 L CNN
 F 1 "0" H 3518 3645 50  0000 L CNN
-F 2 "Resistor_THT:R_Axial_DIN0207_L6.3mm_D2.5mm_P2.54mm_Vertical" V 3490 3680 50  0001 C CNN
+F 2 "Resistor_SMD:R_0805_2012Metric_Pad1.15x1.40mm_HandSolder" V 3490 3680 50  0001 C CNN
 F 3 "~" H 3450 3690 50  0001 C CNN
 	1    3450 3690
@@
 F 0 "JP1" H 3520 3280 50  0000 R CNN
 F 1 "Rest_connect" H 3670 3360 50  0000 R CNN
-F 2 "Jumper:SolderJumper-2_P1.3mm_Open_TrianglePad1.0x1.5mm" H 3450 3230 50  0001 C CNN
+F 2 "Jumper:SolderJumper-2_P1.3mm_Open_RoundedPad1.0x1.5mm" H 3450 3230 50  0001 C CNN
 F 3 "~" H 3450 3230 50  0001 C CNN
 	1    3450 3230
@@
 Text Notes 1960 6170 0    157  ~ 31
 LED to know the status
-$Comp
-L Device:LED_Small_ALT D2
-U 1 1 5EFD7759
-P 2490 7080
-F 0 "D2" V 2536 7010 50  0000 R CNN
-F 1 "LED_data+" V 2445 7010 50  0000 R CNN
-F 2 "LED_THT:LED_D3.0mm_Clear" V 2490 7080 50  0001 C CNN
-F 3 "~" V 2490 7080 50  0001 C CNN
-	1    2490 7080
-	0    -1   -1   0
-$EndComp
-$Comp
-L Device:LED_Small_ALT D3
-U 1 1 5EFD84EB
-P 3330 7080
-F 0 "D3" V 3376 7010 50  0000 R CNN
-F 1 "LED_data-" V 3285 7010 50  0000 R CNN
-F 2 "LED_THT:LED_D3.0mm_Clear" V 3330 7080 50  0001 C CNN
-F 3 "~" V 3330 7080 50  0001 C CNN
-	1    3330 7080
-	0    -1   -1   0
-$EndComp
 $Comp
 L Device:LED_Small_ALT D4
@@
 F 0 "D4" V 4416 7010 50  0000 R CNN
 F 1 "LED_SCK" V 4325 7010 50  0000 R CNN
-F 2 "LED_THT:LED_D3.0mm" V 4370 7080 50  0001 C CNN
+F 2 "LED_SMD:LED_0805_2012Metric_Pad1.15x1.40mm_HandSolder" V 4370 7080 50  0001 C CNN
 F 3 "~" V 4370 7080 50  0001 C CNN
 	1    4370 7080
 	0    -1   -1   0
-$EndComp
-$Comp
-L Device:R_US R2
-U 1 1 5EFD8DF9
-P 2490 6830
-F 0 "R2" H 2558 6876 50  0000 L CNN
-F 1 "1k" H 2558 6785 50  0000 L CNN
-F 2 "Resistor_THT:R_Axial_DIN0207_L6.3mm_D2.5mm_P2.54mm_Vertical" V 2530 6820 50  0001 C CNN
-F 3 "~" H 2490 6830 50  0001 C CNN
-	1    2490 6830
-	1    0    0    -1
-$EndComp
-$Comp
-L Device:R_US R3
-U 1 1 5EFD9C83
-P 3330 6830
-F 0 "R3" H 3398 6876 50  0000 L CNN
-F 1 "1k" H 3398 6785 50  0000 L CNN
-F 2 "Resistor_THT:R_Axial_DIN0207_L6.3mm_D2.5mm_P2.54mm_Vertical" V 3370 6820 50  0001 C CNN
-F 3 "~" H 3330 6830 50  0001 C CNN
-	1    3330 6830
-	1    0    0    -1
 $EndComp
 $Comp
@@
 F 0 "R6" H 4438 6876 50  0000 L CNN
 F 1 "1k" H 4438 6785 50  0000 L CNN
-F 2 "Resistor_THT:R_Axial_DIN0207_L6.3mm_D2.5mm_P2.54mm_Vertical" V 4410 6820 50  0001 C CNN
+F 2 "Resistor_SMD:R_0805_2012Metric_Pad1.15x1.40mm_HandSolder" V 4410 6820 50  0001 C CNN
 F 3 "~" H 4370 6830 50  0001 C CNN
 	1    4370 6830
 	1    0    0    -1
 $EndComp
-Wire Wire Line
-	2490 7180 3330 7180
 Connection ~ 3330 7180
 Wire Wire Line
@@
 $EndComp
 Wire Wire Line
-	2490 6680 2490 6570
-Wire Wire Line
-	3330 6680 3330 6570
-Wire Wire Line
 	4370 6680 4370 6540
-Text Label 2490 6570 0    39   ~ 8
-D+
-Text Label 3330 6570 0    39   ~ 8
-D-
 Text Label 4370 6540 0    39   ~ 8
 SCK
@@
 F 0 "D1" V 1816 7010 50  0000 R CNN
 F 1 "LED_power" V 1725 7010 50  0000 R CNN
-F 2 "LED_THT:LED_D3.0mm" V 1770 7080 50  0001 C CNN
+F 2 "LED_SMD:LED_0805_2012Metric_Pad1.15x1.40mm_HandSolder" V 1770 7080 50  0001 C CNN
 F 3 "~" V 1770 7080 50  0001 C CNN
 	1    1770 7080
@@
 F 0 "R1" H 1838 6876 50  0000 L CNN
 F 1 "1k" H 1838 6785 50  0000 L CNN
-F 2 "Resistor_THT:R_Axial_DIN0207_L6.3mm_D2.5mm_P2.54mm_Vertical" V 1810 6820 50  0001 C CNN
+F 2 "Resistor_SMD:R_0805_2012Metric_Pad1.15x1.40mm_HandSolder" V 1810 6820 50  0001 C CNN
 F 3 "~" H 1770 6830 50  0001 C CNN
 	1    1770 6830
@@
 VCC
 Wire Wire Line
-	1770 7180 2490 7180
-Connection ~ 2490 7180
+	1770 7180 3330 7180
 $EndSCHEMATC
