File: USBTINYISP_MICRO_USB.kicad_pcb (KiCad board)
At the start: 2 copper layers, 17 parts, among them J1 USB_B_Micro, J2 AVR-ISP-6, U1 ATtiny84-20PU, Y1 12MHZ

Commit message: update
Parts:
- removed C1, C2: 18pf, Capacitor_THT:C_Disc_D3.0mm_W1.6mm_P2.50mm
- removed C3: 0.1uf, Capacitor_THT:C_Disc_D3.0mm_W1.6mm_P2.50mm
- removed C4: 10uf, Capacitor_THT:C_Disc_D3.0mm_W1.6mm_P2.50mm
- removed D1, D2: 3v3, Diode_THT:D_DO-15_P2.54mm_Vertical_AnodeUp
- removed J1: USB_B_Micro, Connector_USB:USB_Micro-B_Molex_47346-0001
- removed J2: AVR-ISP-6, Connector_PinHeader_2.54mm:PinHeader_2x03_P2.54mm_Vertical
- removed JP1: Rest_connect, Jumper:SolderJumper-2_P1.3mm_Open_TrianglePad1.0x1.5mm
- removed JP2: USB_power, Jumper:SolderJumper-2_P1.3mm_Bridged2Bar_RoundedPad1.0x1.5mm
- removed R1: 0, Resistor_THT:R_Axial_DIN0204_L3.6mm_D1.6mm_P1.90mm_Vertical
- removed R2: 10k, Resistor_THT:R_Axial_DIN0204_L3.6mm_D1.6mm_P1.90mm_Vertical
- removed R3: 1.5k, Resistor_THT:R_Axial_DIN0204_L3.6mm_D1.6mm_P1.90mm_Vertical
- removed R4, R5: 68, Resistor_THT:R_Axial_DIN0204_L3.6mm_D1.6mm_P1.90mm_Vertical
- removed U1: ATtiny84-20PU, Package_DIP:DIP-14_W7.62mm
- removed Y1: 12MHZ, Crystal:Crystal_HC49-4H_Vertical
Other:
- net class Default: trace_width 0.25 -> 0.4; via_dia 0.8 -> 1.6; via_drill 0.4 -> 1

Commit message: update
Parts:
- added C1: 18pf, Capacitor_THT:C_Disc_D3.0mm_W1.6mm_P2.50mm, F.Cu at (93.5, 110.3)
- added C2: 18pf, Capacitor_THT:C_Disc_D3.0mm_W1.6mm_P2.50mm, F.Cu at (96.1, 110.3)
- added C3: 0.1uf, Capacitor_THT:C_Disc_D3.0mm_W1.6mm_P2.50mm, F.Cu at (74.4, 63.2)
- added C4: 10uf, Capacitor_THT:C_Disc_D3.0mm_W1.6mm_P2.50mm, F.Cu at (88.7, 101.3)
- added D1: LED_power, LED_THT:LED_D3.0mm, F.Cu at (86.0, 50.5)
- added D2: LED_data+, LED_THT:LED_D3.0mm_Clear, F.Cu at (68.6, 64.4)
- added D3: LED_data-, LED_THT:LED_D3.0mm_Clear, F.Cu at (76.2, 54.7)
- added D4: LED_SCK, LED_THT:LED_D3.0mm, F.Cu at (122.9, 89.4)
- added D5: 3v3, Diode_THT:D_DO-41_SOD81_P2.54mm_Vertical_AnodeUp, F.Cu at (80.6, 103.6)
- added D6: 3v3, Diode_THT:D_DO-41_SOD81_P2.54mm_Vertical_AnodeUp, F.Cu at (80.4, 90.5)
- added J1: USB_B_Micro, Connector_USB:USB_Micro-B_Molex_47346-0001, B.Cu at (78.9, 97.0)
- added J2: AVR-ISP-6, Connector_PinHeader_2.54mm:PinHeader_2x03_P2.54mm_Vertical, F.Cu at (116.1, 94.2)
- added JP1: Rest_connect, Jumper:SolderJumper-2_P1.3mm_Open_TrianglePad1.0x1.5mm, B.Cu at (121.7, 79.6)
- added JP2: USB_power, Jumper:SolderJumper-2_P1.3mm_Bridged2Bar_RoundedPad1.0x1.5mm, B.Cu at (122.7, 113.8)
- added R1: 1k, Resistor_THT:R_Axial_DIN0207_L6.3mm_D2.5mm_P2.54mm_Vertical, F.Cu at (67.2, 41.6)
- added R2: 1k, Resistor_THT:R_Axial_DIN0207_L6.3mm_D2.5mm_P2.54mm_Vertical, F.Cu at (55.8, 45.9)
- added R3: 1k, Resistor_THT:R_Axial_DIN0207_L6.3mm_D2.5mm_P2.54mm_Vertical, F.Cu at (66.6, 45.9)
- added R4: 0, Resistor_THT:R_Axial_DIN0207_L6.3mm_D2.5mm_P2.54mm_Vertical, F.Cu at (55.8, 49.9)
- added R5: 10k, Resistor_THT:R_Axial_DIN0207_L6.3mm_D2.5mm_P2.54mm_Vertical, F.Cu at (55.8, 54.0)
- added R6: 1k, Resistor_THT:R_Axial_DIN0207_L6.3mm_D2.5mm_P2.54mm_Vertical, F.Cu at (115.3, 89.4)
- added R7: 1.5k, Resistor_THT:R_Axial_DIN0207_L6.3mm_D2.5mm_P2.54mm_Vertical, F.Cu at (66.6, 49.9)
- added R8: 68, Resistor_THT:R_Axial_DIN0207_L6.3mm_D2.5mm_P2.54mm_Vertical, F.Cu at (77.9, 41.6)
- added R9: 68, Resistor_THT:R_Axial_DIN0207_L6.3mm_D2.5mm_P2.54mm_Vertical, F.Cu at (86.1, 92.9)
- added U1: ATtiny84-20PU, Package_DIP:DIP-14_W7.62mm, F.Cu at (91.1, 101.2)
- added Y1: 12MHZ, Crystal:Crystal_HC49-4H_Vertical, F.Cu at (92.4, 105.7)
Routing:
- net Net-(JP1-Pad2): track 0.00 -> 39.9 mm
- net /SCK: track 0.00 -> 26.9 mm
- net /D+: track 0.00 -> 25.3 mm
- net /MOSI: track 0.00 -> 17.9 mm
- net /RST: track 0.00 -> 17.2 mm
- net /VCC: track 0.00 -> 12.0 mm
- net Net-(D6-Pad1): track 0.00 -> 12.0 mm
- net /MISO: track 0.00 -> 10.0 mm
- net Net-(D5-Pad1): track 0.00 -> 7.75 mm
- net Net-(C1-Pad2): track 0.00 -> 7.59 mm
- net Net-(C2-Pad2): track 0.00 -> 7.50 mm
- net Net-(D4-Pad2): track 0.00 -> 2.48 mm
- net GND: track 0.00 -> 1.19 mm
- added copper zone on B.Cu, net GND
Other:
- board outline added: 49.8 x 39.7 mm
- net class Default: clearance 0.2 -> 0.25; trace_width 0.4 -> 0.39
- rule trace_clearance: 0.2 -> 0.25

Commit message: update
Parts:
- C1, C2, C3, C4: footprint Capacitor_THT:C_Disc_D3.0mm_W1.6mm_P2.50mm -> Capacitor_SMD:C_0805_2012Metric_Pad1.15x1.40mm_HandSolder
- D1, D4: footprint LED_THT:LED_D3.0mm -> LED_SMD:LED_0805_2012Metric_Pad1.15x1.40mm_HandSolder
- D2, D3: footprint LED_THT:LED_D3.0mm_Clear -> LED_SMD:LED_0805_2012Metric_Pad1.15x1.40mm_HandSolder
- D5, D6: footprint Diode_THT:D_DO-41_SOD81_P2.54mm_Vertical_AnodeUp -> Diode_SMD:D_0805_2012Metric_Pad1.15x1.40mm_HandSolder
- J1, JP2: moved to F.Cu
- J2: footprint Connector_PinHeader_2.54mm:PinHeader_2x03_P2.54mm_Vertical -> Connector_PinHeader_2.54mm:PinHeader_2x03_P2.54mm_Vertical_SMD
- JP1: footprint Jumper:SolderJumper-2_P1.3mm_Open_TrianglePad1.0x1.5mm -> Jumper:SolderJumper-2_P1.3mm_Open_RoundedPad1.0x1.5mm; moved to F.Cu
- R1, R2, R3, R4, R5, R6, R7, R8, R9: footprint Resistor_THT:R_Axial_DIN0207_L6.3mm_D2.5mm_P2.54mm_Vertical -> Resistor_SMD:R_0805_2012Metric_Pad1.15x1.40mm_HandSolder
- U1: footprint Package_DIP:DIP-14_W7.62mm -> Package_SO:SOIC-14_3.9x8.7mm_P1.27mm
- Y1: footprint Crystal:Crystal_HC49-4H_Vertical -> Crystal:Crystal_SMD_HC49-SD
- moved D4 63.5 mm to (66.0, 61.4), turned to 0 degrees
- moved R6 53.3 mm to (70.1, 61.4), turned to 180 degrees
- moved D3 52.9 mm to (26.6, 36.2)
- moved JP1 52.3 mm to (69.8, 72.9), turned to 180 degrees
- moved D2 50.2 mm to (38.5, 24.3)
- moved JP2 50.0 mm to (81.7, 85.2)
- moved C4 48.1 mm to (49.9, 72.8)
- moved J2 47.5 mm to (78.7, 65.0)
- moved D5 46.5 mm to (51.7, 67.2), turned to 0 degrees
- moved J1 42.9 mm to (43.4, 72.9), turned to 270 degrees
- moved U1 42.6 mm to (65.0, 67.6)
- moved C1 38.4 mm to (67.0, 82.5), turned to 180 degrees
- moved R8 38.3 mm to (48.5, 66.2), turned to 270 degrees
- moved Y1 36.9 mm to (68.0, 78.1)
- moved C2 36.8 mm to (72.0, 82.5), turned to 0 degrees
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Routing:
- net /VCC: track 12.0 -> 72.5 mm
- net GND: track 1.19 -> 57.0 mm
- net Net-(J2-Pad2): track 0.00 -> 25.6 mm
- net Net-(JP1-Pad2): track 39.9 -> 17.7 mm
- net /D-: track 0.00 -> 17.1 mm
- net /D+: track 25.3 -> 13.2 mm
- net /SCK: track 26.9 -> 16.1 mm
- net Net-(C2-Pad2): track 7.50 -> 18.2 mm
- net Net-(C1-Pad2): track 7.59 -> 13.9 mm
- net Net-(D5-Pad1): track 7.75 -> 13.8 mm
- net Net-(JP1-Pad1): track 0.00 -> 5.67 mm
- net /RST: track 17.2 -> 14.2 mm
- net Net-(D6-Pad1): track 12.0 -> 14.8 mm
- net Net-(D1-Pad2): track 0.00 -> 1.94 mm
- net /MISO: track 10.0 -> 8.45 mm
- added copper zone on F.Cu, net GND
- removed copper zone on B.Cu, net GND
Other:
- board size 49.8 x 39.7 mm -> 44.8 x 29 mm

Commit message: update
Parts:
- removed D2: LED_data+, LED_SMD:LED_0805_2012Metric_Pad1.15x1.40mm_HandSolder
- removed D3: LED_data-, LED_SMD:LED_0805_2012Metric_Pad1.15x1.40mm_HandSolder
- removed R2, R3: 1k, Resistor_SMD:R_0805_2012Metric_Pad1.15x1.40mm_HandSolder
- added C1: 18pf, Capacitor_SMD:C_0805_2012Metric_Pad1.15x1.40mm_HandSolder, F.Cu at (142.9, 160.6)
- added C1: 18pf, Capacitor_SMD:C_0805_2012Metric_Pad1.15x1.40mm_HandSolder, F.Cu at (92.1, 130.1)
- added C1: 18pf, Capacitor_SMD:C_0805_2012Metric_Pad1.15x1.40mm_HandSolder, F.Cu at (142.9, 99.6)
- added C1: 18pf, Capacitor_SMD:C_0805_2012Metric_Pad1.15x1.40mm_HandSolder, F.Cu at (244.5, 99.6)
- added C1: 18pf, Capacitor_SMD:C_0805_2012Metric_Pad1.15x1.40mm_HandSolder, F.Cu at (193.7, 99.6)
- added C1: 18pf, Capacitor_SMD:C_0805_2012Metric_Pad1.15x1.40mm_HandSolder, F.Cu at (41.3, 99.6)
- added C1: 18pf, Capacitor_SMD:C_0805_2012Metric_Pad1.15x1.40mm_HandSolder, F.Cu at (92.1, 99.6)
- added C1: 18pf, Capacitor_SMD:C_0805_2012Metric_Pad1.15x1.40mm_HandSolder, F.Cu at (142.9, 69.2)
- added C1: 18pf, Capacitor_SMD:C_0805_2012Metric_Pad1.15x1.40mm_HandSolder, F.Cu at (193.7, 69.2)
- added C1: 18pf, Capacitor_SMD:C_0805_2012Metric_Pad1.15x1.40mm_HandSolder, F.Cu at (244.5, 69.2)
- added C1: 18pf, Capacitor_SMD:C_0805_2012Metric_Pad1.15x1.40mm_HandSolder, F.Cu at (41.3, 69.2)
- added C1: 18pf, Capacitor_SMD:C_0805_2012Metric_Pad1.15x1.40mm_HandSolder, F.Cu at (193.7, 160.6)
- added C1: 18pf, Capacitor_SMD:C_0805_2012Metric_Pad1.15x1.40mm_HandSolder, F.Cu at (92.1, 69.2)
- added C1: 18pf, Capacitor_SMD:C_0805_2012Metric_Pad1.15x1.40mm_HandSolder, F.Cu at (244.5, 38.7)
- added C1: 18pf, Capacitor_SMD:C_0805_2012Metric_Pad1.15x1.40mm_HandSolder, F.Cu at (193.7, 38.7)
- added C1: 18pf, Capacitor_SMD:C_0805_2012Metric_Pad1.15x1.40mm_HandSolder, F.Cu at (142.9, 38.7)
- added C1: 18pf, Capacitor_SMD:C_0805_2012Metric_Pad1.15x1.40mm_HandSolder, F.Cu at (92.1, 38.7)
- added C1: 18pf, Capacitor_SMD:C_0805_2012Metric_Pad1.15x1.40mm_HandSolder, F.Cu at (41.3, 160.6)
- added C1: 18pf, Capacitor_SMD:C_0805_2012Metric_Pad1.15x1.40mm_HandSolder, F.Cu at (244.5, 160.6)
- added C1: 18pf, Capacitor_SMD:C_0805_2012Metric_Pad1.15x1.40mm_HandSolder, F.Cu at (92.1, 160.6)
- added C1: 18pf, Capacitor_SMD:C_0805_2012Metric_Pad1.15x1.40mm_HandSolder, F.Cu at (142.9, 130.1)
- added C1: 18pf, Capacitor_SMD:C_0805_2012Metric_Pad1.15x1.40mm_HandSolder, F.Cu at (41.3, 130.1)
- added C1: 18pf, Capacitor_SMD:C_0805_2012Metric_Pad1.15x1.40mm_HandSolder, F.Cu at (244.5, 130.1)
- added C1: 18pf, Capacitor_SMD:C_0805_2012Metric_Pad1.15x1.40mm_HandSolder, F.Cu at (193.7, 130.1)
- added C2: 18pf, Capacitor_SMD:C_0805_2012Metric_Pad1.15x1.40mm_HandSolder, F.Cu at (147.8, 160.6)
- added C2: 18pf, Capacitor_SMD:C_0805_2012Metric_Pad1.15x1.40mm_HandSolder, F.Cu at (97.0, 130.1)
- added C2: 18pf, Capacitor_SMD:C_0805_2012Metric_Pad1.15x1.40mm_HandSolder, F.Cu at (147.8, 99.6)
- added C2: 18pf, Capacitor_SMD:C_0805_2012Metric_Pad1.15x1.40mm_HandSolder, F.Cu at (249.4, 99.6)
- added C2: 18pf, Capacitor_SMD:C_0805_2012Metric_Pad1.15x1.40mm_HandSolder, F.Cu at (198.7, 99.6)
- added C2: 18pf, Capacitor_SMD:C_0805_2012Metric_Pad1.15x1.40mm_HandSolder, F.Cu at (46.2, 99.6)
- added C2: 18pf, Capacitor_SMD:C_0805_2012Metric_Pad1.15x1.40mm_HandSolder, F.Cu at (97.0, 99.6)
- added C2: 18pf, Capacitor_SMD:C_0805_2012Metric_Pad1.15x1.40mm_HandSolder, F.Cu at (147.8, 69.2)
- added C2: 18pf, Capacitor_SMD:C_0805_2012Metric_Pad1.15x1.40mm_HandSolder, F.Cu at (198.7, 69.2)
- added C2: 18pf, Capacitor_SMD:C_0805_2012Metric_Pad1.15x1.40mm_HandSolder, F.Cu at (249.4, 69.2)
- added C2: 18pf, Capacitor_SMD:C_0805_2012Metric_Pad1.15x1.40mm_HandSolder, F.Cu at (46.2, 69.2)
- added C2: 18pf, Capacitor_SMD:C_0805_2012Metric_Pad1.15x1.40mm_HandSolder, F.Cu at (249.4, 160.6)
- added C2: 18pf, Capacitor_SMD:C_0805_2012Metric_Pad1.15x1.40mm_HandSolder, F.Cu at (97.0, 69.2)
- added C2: 18pf, Capacitor_SMD:C_0805_2012Metric_Pad1.15x1.40mm_HandSolder, F.Cu at (249.4, 38.7)
- added C2: 18pf, Capacitor_SMD:C_0805_2012Metric_Pad1.15x1.40mm_HandSolder, F.Cu at (198.7, 38.7)
- added C2: 18pf, Capacitor_SMD:C_0805_2012Metric_Pad1.15x1.40mm_HandSolder, F.Cu at (147.8, 38.7)
- added C2: 18pf, Capacitor_SMD:C_0805_2012Metric_Pad1.15x1.40mm_HandSolder, F.Cu at (97.0, 38.7)
- added C2: 18pf, Capacitor_SMD:C_0805_2012Metric_Pad1.15x1.40mm_HandSolder, F.Cu at (198.7, 160.6)
- added C2: 18pf, Capacitor_SMD:C_0805_2012Metric_Pad1.15x1.40mm_HandSolder, F.Cu at (46.2, 160.6)
- added C2: 18pf, Capacitor_SMD:C_0805_2012Metric_Pad1.15x1.40mm_HandSolder, F.Cu at (97.0, 160.6)
- added C2: 18pf, Capacitor_SMD:C_0805_2012Metric_Pad1.15x1.40mm_HandSolder, F.Cu at (147.8, 130.1)
- added C2: 18pf, Capacitor_SMD:C_0805_2012Metric_Pad1.15x1.40mm_HandSolder, F.Cu at (249.4, 130.1)
- added C2: 18pf, Capacitor_SMD:C_0805_2012Metric_Pad1.15x1.40mm_HandSolder, F.Cu at (198.7, 130.1)
- added C2: 18pf, Capacitor_SMD:C_0805_2012Metric_Pad1.15x1.40mm_HandSolder, F.Cu at (46.2, 130.1)
- added C3: 0.1uf, Capacitor_SMD:C_0805_2012Metric_Pad1.15x1.40mm_HandSolder, F.Cu at (127.9, 148.6)
- added C3: 0.1uf, Capacitor_SMD:C_0805_2012Metric_Pad1.15x1.40mm_HandSolder, F.Cu at (77.1, 118.1)
- added C3: 0.1uf, Capacitor_SMD:C_0805_2012Metric_Pad1.15x1.40mm_HandSolder, F.Cu at (127.9, 87.7)
- added C3: 0.1uf, Capacitor_SMD:C_0805_2012Metric_Pad1.15x1.40mm_HandSolder, F.Cu at (229.5, 87.7)
- added C3: 0.1uf, Capacitor_SMD:C_0805_2012Metric_Pad1.15x1.40mm_HandSolder, F.Cu at (178.7, 87.7)
- added C3: 0.1uf, Capacitor_SMD:C_0805_2012Metric_Pad1.15x1.40mm_HandSolder, F.Cu at (26.3, 87.7)
- added C3: 0.1uf, Capacitor_SMD:C_0805_2012Metric_Pad1.15x1.40mm_HandSolder, F.Cu at (77.1, 87.7)
- added C3: 0.1uf, Capacitor_SMD:C_0805_2012Metric_Pad1.15x1.40mm_HandSolder, F.Cu at (127.9, 57.2)
- added C3: 0.1uf, Capacitor_SMD:C_0805_2012Metric_Pad1.15x1.40mm_HandSolder, F.Cu at (178.7, 57.2)
- added C3: 0.1uf, Capacitor_SMD:C_0805_2012Metric_Pad1.15x1.40mm_HandSolder, F.Cu at (229.5, 57.2)
- added C3: 0.1uf, Capacitor_SMD:C_0805_2012Metric_Pad1.15x1.40mm_HandSolder, F.Cu at (26.3, 57.2)
- added C3: 0.1uf, Capacitor_SMD:C_0805_2012Metric_Pad1.15x1.40mm_HandSolder, F.Cu at (229.5, 148.6)
- added C3: 0.1uf, Capacitor_SMD:C_0805_2012Metric_Pad1.15x1.40mm_HandSolder, F.Cu at (77.1, 57.2)
- added C3: 0.1uf, Capacitor_SMD:C_0805_2012Metric_Pad1.15x1.40mm_HandSolder, F.Cu at (229.5, 26.7)
- added C3: 0.1uf, Capacitor_SMD:C_0805_2012Metric_Pad1.15x1.40mm_HandSolder, F.Cu at (178.7, 26.7)
- added C3: 0.1uf, Capacitor_SMD:C_0805_2012Metric_Pad1.15x1.40mm_HandSolder, F.Cu at (127.9, 26.7)
- added C3: 0.1uf, Capacitor_SMD:C_0805_2012Metric_Pad1.15x1.40mm_HandSolder, F.Cu at (77.1, 26.7)
- added C3: 0.1uf, Capacitor_SMD:C_0805_2012Metric_Pad1.15x1.40mm_HandSolder, F.Cu at (178.7, 148.6)
- added C3: 0.1uf, Capacitor_SMD:C_0805_2012Metric_Pad1.15x1.40mm_HandSolder, F.Cu at (26.3, 148.6)
- added C3: 0.1uf, Capacitor_SMD:C_0805_2012Metric_Pad1.15x1.40mm_HandSolder, F.Cu at (77.1, 148.6)
- added C3: 0.1uf, Capacitor_SMD:C_0805_2012Metric_Pad1.15x1.40mm_HandSolder, F.Cu at (127.9, 118.1)
- added C3: 0.1uf, Capacitor_SMD:C_0805_2012Metric_Pad1.15x1.40mm_HandSolder, F.Cu at (229.5, 118.1)
- added C3: 0.1uf, Capacitor_SMD:C_0805_2012Metric_Pad1.15x1.40mm_HandSolder, F.Cu at (178.7, 118.1)
- added C3: 0.1uf, Capacitor_SMD:C_0805_2012Metric_Pad1.15x1.40mm_HandSolder, F.Cu at (26.3, 118.1)
- added C4: 10uf, Capacitor_SMD:C_0805_2012Metric_Pad1.15x1.40mm_HandSolder, F.Cu at (125.8, 150.9)
- added C4: 10uf, Capacitor_SMD:C_0805_2012Metric_Pad1.15x1.40mm_HandSolder, F.Cu at (75.0, 120.4)
- added C4: 10uf, Capacitor_SMD:C_0805_2012Metric_Pad1.15x1.40mm_HandSolder, F.Cu at (125.8, 89.9)
- added C4: 10uf, Capacitor_SMD:C_0805_2012Metric_Pad1.15x1.40mm_HandSolder, F.Cu at (176.6, 89.9)
- added C4: 10uf, Capacitor_SMD:C_0805_2012Metric_Pad1.15x1.40mm_HandSolder, F.Cu at (227.4, 89.9)
- added C4: 10uf, Capacitor_SMD:C_0805_2012Metric_Pad1.15x1.40mm_HandSolder, F.Cu at (24.2, 89.9)
- added C4: 10uf, Capacitor_SMD:C_0805_2012Metric_Pad1.15x1.40mm_HandSolder, F.Cu at (75.0, 89.9)
- added C4: 10uf, Capacitor_SMD:C_0805_2012Metric_Pad1.15x1.40mm_HandSolder, F.Cu at (125.8, 59.5)
- added C4: 10uf, Capacitor_SMD:C_0805_2012Metric_Pad1.15x1.40mm_HandSolder, F.Cu at (176.6, 59.5)
- added C4: 10uf, Capacitor_SMD:C_0805_2012Metric_Pad1.15x1.40mm_HandSolder, F.Cu at (227.4, 59.5)
- added C4: 10uf, Capacitor_SMD:C_0805_2012Metric_Pad1.15x1.40mm_HandSolder, F.Cu at (24.2, 59.5)
- added C4: 10uf, Capacitor_SMD:C_0805_2012Metric_Pad1.15x1.40mm_HandSolder, F.Cu at (176.6, 150.9)
- added C4: 10uf, Capacitor_SMD:C_0805_2012Metric_Pad1.15x1.40mm_HandSolder, F.Cu at (75.0, 59.5)
- added C4: 10uf, Capacitor_SMD:C_0805_2012Metric_Pad1.15x1.40mm_HandSolder, F.Cu at (227.4, 29.0)
- added C4: 10uf, Capacitor_SMD:C_0805_2012Metric_Pad1.15x1.40mm_HandSolder, F.Cu at (176.6, 29.0)
- added C4: 10uf, Capacitor_SMD:C_0805_2012Metric_Pad1.15x1.40mm_HandSolder, F.Cu at (125.8, 29.0)
- added C4: 10uf, Capacitor_SMD:C_0805_2012Metric_Pad1.15x1.40mm_HandSolder, F.Cu at (75.0, 29.0)
- added C4: 10uf, Capacitor_SMD:C_0805_2012Metric_Pad1.15x1.40mm_HandSolder, F.Cu at (227.4, 150.9)
- added C4: 10uf, Capacitor_SMD:C_0805_2012Metric_Pad1.15x1.40mm_HandSolder, F.Cu at (24.2, 150.9)
- added C4: 10uf, Capacitor_SMD:C_0805_2012Metric_Pad1.15x1.40mm_HandSolder, F.Cu at (75.0, 150.9)
- added C4: 10uf, Capacitor_SMD:C_0805_2012Metric_Pad1.15x1.40mm_HandSolder, F.Cu at (125.8, 120.4)
- added C4: 10uf, Capacitor_SMD:C_0805_2012Metric_Pad1.15x1.40mm_HandSolder, F.Cu at (176.6, 120.4)
- added C4: 10uf, Capacitor_SMD:C_0805_2012Metric_Pad1.15x1.40mm_HandSolder, F.Cu at (227.4, 120.4)
- added C4: 10uf, Capacitor_SMD:C_0805_2012Metric_Pad1.15x1.40mm_HandSolder, F.Cu at (24.2, 120.4)
- added D1: LED_power, LED_SMD:LED_0805_2012Metric_Pad1.15x1.40mm_HandSolder, F.Cu at (128.6, 142.9)
- added D1: LED_power, LED_SMD:LED_0805_2012Metric_Pad1.15x1.40mm_HandSolder, F.Cu at (27.0, 112.4)
- added D1: LED_power, LED_SMD:LED_0805_2012Metric_Pad1.15x1.40mm_HandSolder, F.Cu at (128.6, 81.9)
- added D1: LED_power, LED_SMD:LED_0805_2012Metric_Pad1.15x1.40mm_HandSolder, F.Cu at (179.4, 81.9)
- added D1: LED_power, LED_SMD:LED_0805_2012Metric_Pad1.15x1.40mm_HandSolder, F.Cu at (77.8, 81.9)
- added D1: LED_power, LED_SMD:LED_0805_2012Metric_Pad1.15x1.40mm_HandSolder, F.Cu at (230.2, 81.9)
- added D1: LED_power, LED_SMD:LED_0805_2012Metric_Pad1.15x1.40mm_HandSolder, F.Cu at (27.0, 81.9)
- added D1: LED_power, LED_SMD:LED_0805_2012Metric_Pad1.15x1.40mm_HandSolder, F.Cu at (128.6, 51.4)
- added D1: LED_power, LED_SMD:LED_0805_2012Metric_Pad1.15x1.40mm_HandSolder, F.Cu at (179.4, 51.4)
- added D1: LED_power, LED_SMD:LED_0805_2012Metric_Pad1.15x1.40mm_HandSolder, F.Cu at (230.2, 51.4)
- added D1: LED_power, LED_SMD:LED_0805_2012Metric_Pad1.15x1.40mm_HandSolder, F.Cu at (27.0, 51.4)
- added D1: LED_power, LED_SMD:LED_0805_2012Metric_Pad1.15x1.40mm_HandSolder, F.Cu at (77.8, 142.9)
- added D1: LED_power, LED_SMD:LED_0805_2012Metric_Pad1.15x1.40mm_HandSolder, F.Cu at (77.8, 51.4)
- added D1: LED_power, LED_SMD:LED_0805_2012Metric_Pad1.15x1.40mm_HandSolder, F.Cu at (230.2, 20.9)
- added D1: LED_power, LED_SMD:LED_0805_2012Metric_Pad1.15x1.40mm_HandSolder, F.Cu at (179.4, 20.9)
- added D1: LED_power, LED_SMD:LED_0805_2012Metric_Pad1.15x1.40mm_HandSolder, F.Cu at (128.6, 20.9)
- added D1: LED_power, LED_SMD:LED_0805_2012Metric_Pad1.15x1.40mm_HandSolder, F.Cu at (77.8, 20.9)
- added D1: LED_power, LED_SMD:LED_0805_2012Metric_Pad1.15x1.40mm_HandSolder, F.Cu at (179.4, 142.9)
- added D1: LED_power, LED_SMD:LED_0805_2012Metric_Pad1.15x1.40mm_HandSolder, F.Cu at (230.2, 142.9)
- added D1: LED_power, LED_SMD:LED_0805_2012Metric_Pad1.15x1.40mm_HandSolder, F.Cu at (27.0, 142.9)
- added D1: LED_power, LED_SMD:LED_0805_2012Metric_Pad1.15x1.40mm_HandSolder, F.Cu at (128.6, 112.4)
- added D1: LED_power, LED_SMD:LED_0805_2012Metric_Pad1.15x1.40mm_HandSolder, F.Cu at (77.8, 112.4)
- added D1: LED_power, LED_SMD:LED_0805_2012Metric_Pad1.15x1.40mm_HandSolder, F.Cu at (179.4, 112.4)
- added D1: LED_power, LED_SMD:LED_0805_2012Metric_Pad1.15x1.40mm_HandSolder, F.Cu at (230.2, 112.4)
- added D4: LED_SCK, LED_SMD:LED_0805_2012Metric_Pad1.15x1.40mm_HandSolder, F.Cu at (141.8, 139.4)
- added D4: LED_SCK, LED_SMD:LED_0805_2012Metric_Pad1.15x1.40mm_HandSolder, F.Cu at (91.0, 109.0)
- added D4: LED_SCK, LED_SMD:LED_0805_2012Metric_Pad1.15x1.40mm_HandSolder, F.Cu at (141.8, 78.5)
- added D4: LED_SCK, LED_SMD:LED_0805_2012Metric_Pad1.15x1.40mm_HandSolder, F.Cu at (192.6, 78.5)
- added D4: LED_SCK, LED_SMD:LED_0805_2012Metric_Pad1.15x1.40mm_HandSolder, F.Cu at (243.4, 78.5)
- added D4: LED_SCK, LED_SMD:LED_0805_2012Metric_Pad1.15x1.40mm_HandSolder, F.Cu at (40.2, 78.5)
- added D4: LED_SCK, LED_SMD:LED_0805_2012Metric_Pad1.15x1.40mm_HandSolder, F.Cu at (91.0, 78.5)
- added D4: LED_SCK, LED_SMD:LED_0805_2012Metric_Pad1.15x1.40mm_HandSolder, F.Cu at (141.8, 48.0)
- added D4: LED_SCK, LED_SMD:LED_0805_2012Metric_Pad1.15x1.40mm_HandSolder, F.Cu at (192.6, 48.0)
- added D4: LED_SCK, LED_SMD:LED_0805_2012Metric_Pad1.15x1.40mm_HandSolder, F.Cu at (243.4, 48.0)
- added D4: LED_SCK, LED_SMD:LED_0805_2012Metric_Pad1.15x1.40mm_HandSolder, F.Cu at (40.2, 48.0)
- added D4: LED_SCK, LED_SMD:LED_0805_2012Metric_Pad1.15x1.40mm_HandSolder, F.Cu at (192.6, 139.4)
- added D4: LED_SCK, LED_SMD:LED_0805_2012Metric_Pad1.15x1.40mm_HandSolder, F.Cu at (91.0, 48.0)
- added D4: LED_SCK, LED_SMD:LED_0805_2012Metric_Pad1.15x1.40mm_HandSolder, F.Cu at (243.4, 17.5)
- added D4: LED_SCK, LED_SMD:LED_0805_2012Metric_Pad1.15x1.40mm_HandSolder, F.Cu at (192.6, 17.5)
- added D4: LED_SCK, LED_SMD:LED_0805_2012Metric_Pad1.15x1.40mm_HandSolder, F.Cu at (141.8, 17.5)
- added D4: LED_SCK, LED_SMD:LED_0805_2012Metric_Pad1.15x1.40mm_HandSolder, F.Cu at (91.0, 17.5)
- added D4: LED_SCK, LED_SMD:LED_0805_2012Metric_Pad1.15x1.40mm_HandSolder, F.Cu at (243.4, 139.4)
- added D4: LED_SCK, LED_SMD:LED_0805_2012Metric_Pad1.15x1.40mm_HandSolder, F.Cu at (40.2, 139.4)
- added D4: LED_SCK, LED_SMD:LED_0805_2012Metric_Pad1.15x1.40mm_HandSolder, F.Cu at (91.0, 139.4)
- added D4: LED_SCK, LED_SMD:LED_0805_2012Metric_Pad1.15x1.40mm_HandSolder, F.Cu at (141.8, 109.0)
- added D4: LED_SCK, LED_SMD:LED_0805_2012Metric_Pad1.15x1.40mm_HandSolder, F.Cu at (192.6, 109.0)
- added D4: LED_SCK, LED_SMD:LED_0805_2012Metric_Pad1.15x1.40mm_HandSolder, F.Cu at (243.4, 109.0)
- added D4: LED_SCK, LED_SMD:LED_0805_2012Metric_Pad1.15x1.40mm_HandSolder, F.Cu at (40.2, 109.0)
- added D5: 3v3, Diode_SMD:D_0805_2012Metric_Pad1.15x1.40mm_HandSolder, F.Cu at (127.6, 145.3)
- added D5: 3v3, Diode_SMD:D_0805_2012Metric_Pad1.15x1.40mm_HandSolder, F.Cu at (76.8, 114.8)
- added D5: 3v3, Diode_SMD:D_0805_2012Metric_Pad1.15x1.40mm_HandSolder, F.Cu at (127.6, 84.3)
- added D5: 3v3, Diode_SMD:D_0805_2012Metric_Pad1.15x1.40mm_HandSolder, F.Cu at (178.4, 84.3)
- added D5: 3v3, Diode_SMD:D_0805_2012Metric_Pad1.15x1.40mm_HandSolder, F.Cu at (229.2, 84.3)
- added D5: 3v3, Diode_SMD:D_0805_2012Metric_Pad1.15x1.40mm_HandSolder, F.Cu at (26.0, 84.3)
- added D5: 3v3, Diode_SMD:D_0805_2012Metric_Pad1.15x1.40mm_HandSolder, F.Cu at (76.8, 84.3)
- added D5: 3v3, Diode_SMD:D_0805_2012Metric_Pad1.15x1.40mm_HandSolder, F.Cu at (127.6, 53.8)
- added D5: 3v3, Diode_SMD:D_0805_2012Metric_Pad1.15x1.40mm_HandSolder, F.Cu at (178.4, 53.8)
- added D5: 3v3, Diode_SMD:D_0805_2012Metric_Pad1.15x1.40mm_HandSolder, F.Cu at (229.2, 53.8)
- added D5: 3v3, Diode_SMD:D_0805_2012Metric_Pad1.15x1.40mm_HandSolder, F.Cu at (26.0, 53.8)
- added D5: 3v3, Diode_SMD:D_0805_2012Metric_Pad1.15x1.40mm_HandSolder, F.Cu at (178.4, 145.3)
- added D5: 3v3, Diode_SMD:D_0805_2012Metric_Pad1.15x1.40mm_HandSolder, F.Cu at (76.8, 53.8)
- added D5: 3v3, Diode_SMD:D_0805_2012Metric_Pad1.15x1.40mm_HandSolder, F.Cu at (229.2, 23.4)
- added D5: 3v3, Diode_SMD:D_0805_2012Metric_Pad1.15x1.40mm_HandSolder, F.Cu at (178.4, 23.4)
- added D5: 3v3, Diode_SMD:D_0805_2012Metric_Pad1.15x1.40mm_HandSolder, F.Cu at (127.6, 23.4)
- added D5: 3v3, Diode_SMD:D_0805_2012Metric_Pad1.15x1.40mm_HandSolder, F.Cu at (76.8, 23.4)
- added D5: 3v3, Diode_SMD:D_0805_2012Metric_Pad1.15x1.40mm_HandSolder, F.Cu at (229.2, 145.3)
- added D5: 3v3, Diode_SMD:D_0805_2012Metric_Pad1.15x1.40mm_HandSolder, F.Cu at (26.0, 145.3)
- added D5: 3v3, Diode_SMD:D_0805_2012Metric_Pad1.15x1.40mm_HandSolder, F.Cu at (76.8, 145.3)
- added D5: 3v3, Diode_SMD:D_0805_2012Metric_Pad1.15x1.40mm_HandSolder, F.Cu at (127.6, 114.8)
- added D5: 3v3, Diode_SMD:D_0805_2012Metric_Pad1.15x1.40mm_HandSolder, F.Cu at (178.4, 114.8)
- added D5: 3v3, Diode_SMD:D_0805_2012Metric_Pad1.15x1.40mm_HandSolder, F.Cu at (229.2, 114.8)
- added D5: 3v3, Diode_SMD:D_0805_2012Metric_Pad1.15x1.40mm_HandSolder, F.Cu at (26.0, 114.8)
- added D6: 3v3, Diode_SMD:D_0805_2012Metric_Pad1.15x1.40mm_HandSolder, F.Cu at (130.4, 153.6)
- added D6: 3v3, Diode_SMD:D_0805_2012Metric_Pad1.15x1.40mm_HandSolder, F.Cu at (79.6, 123.1)
- added D6: 3v3, Diode_SMD:D_0805_2012Metric_Pad1.15x1.40mm_HandSolder, F.Cu at (130.4, 92.6)
- added D6: 3v3, Diode_SMD:D_0805_2012Metric_Pad1.15x1.40mm_HandSolder, F.Cu at (232.0, 92.6)
- added D6: 3v3, Diode_SMD:D_0805_2012Metric_Pad1.15x1.40mm_HandSolder, F.Cu at (181.2, 92.6)
- added D6: 3v3, Diode_SMD:D_0805_2012Metric_Pad1.15x1.40mm_HandSolder, F.Cu at (28.8, 92.6)
- added D6: 3v3, Diode_SMD:D_0805_2012Metric_Pad1.15x1.40mm_HandSolder, F.Cu at (79.6, 92.6)
- added D6: 3v3, Diode_SMD:D_0805_2012Metric_Pad1.15x1.40mm_HandSolder, F.Cu at (130.4, 62.2)
- added D6: 3v3, Diode_SMD:D_0805_2012Metric_Pad1.15x1.40mm_HandSolder, F.Cu at (181.2, 62.2)
- added D6: 3v3, Diode_SMD:D_0805_2012Metric_Pad1.15x1.40mm_HandSolder, F.Cu at (232.0, 62.2)
- added D6: 3v3, Diode_SMD:D_0805_2012Metric_Pad1.15x1.40mm_HandSolder, F.Cu at (28.8, 62.2)
- added D6: 3v3, Diode_SMD:D_0805_2012Metric_Pad1.15x1.40mm_HandSolder, F.Cu at (232.0, 153.6)
- added D6: 3v3, Diode_SMD:D_0805_2012Metric_Pad1.15x1.40mm_HandSolder, F.Cu at (79.6, 62.2)
- added D6: 3v3, Diode_SMD:D_0805_2012Metric_Pad1.15x1.40mm_HandSolder, F.Cu at (232.0, 31.7)
- added D6: 3v3, Diode_SMD:D_0805_2012Metric_Pad1.15x1.40mm_HandSolder, F.Cu at (181.2, 31.7)
- added D6: 3v3, Diode_SMD:D_0805_2012Metric_Pad1.15x1.40mm_HandSolder, F.Cu at (130.4, 31.7)
- added D6: 3v3, Diode_SMD:D_0805_2012Metric_Pad1.15x1.40mm_HandSolder, F.Cu at (79.6, 31.7)
- added D6: 3v3, Diode_SMD:D_0805_2012Metric_Pad1.15x1.40mm_HandSolder, F.Cu at (181.2, 153.6)
- added D6: 3v3, Diode_SMD:D_0805_2012Metric_Pad1.15x1.40mm_HandSolder, F.Cu at (28.8, 153.6)
- added D6: 3v3, Diode_SMD:D_0805_2012Metric_Pad1.15x1.40mm_HandSolder, F.Cu at (79.6, 153.6)
- added D6: 3v3, Diode_SMD:D_0805_2012Metric_Pad1.15x1.40mm_HandSolder, F.Cu at (130.4, 123.1)
- added D6: 3v3, Diode_SMD:D_0805_2012Metric_Pad1.15x1.40mm_HandSolder, F.Cu at (232.0, 123.1)
- added D6: 3v3, Diode_SMD:D_0805_2012Metric_Pad1.15x1.40mm_HandSolder, F.Cu at (28.8, 123.1)
- added D6: 3v3, Diode_SMD:D_0805_2012Metric_Pad1.15x1.40mm_HandSolder, F.Cu at (181.2, 123.1)
- added G***: LOGO, ved:ved1, F.Cu at (18.4, 163.8)
- added G***: LOGO, ved:ved1, F.Cu at (18.4, 133.3)
- added G***: LOGO, ved:ved1, F.Cu at (18.4, 102.8)
- added G***: LOGO, ved:ved1, F.Cu at (18.4, 72.3)
- added G***: LOGO, ved:ved1, F.Cu at (18.4, 41.9)
- added J1: USB_B_Micro, Connector_USB:USB_Micro-B_Molex_47346-0001, F.Cu at (119.3, 151.0)
- added J1: USB_B_Micro, Connector_USB:USB_Micro-B_Molex_47346-0001, F.Cu at (68.5, 120.5)
- added J1: USB_B_Micro, Connector_USB:USB_Micro-B_Molex_47346-0001, F.Cu at (119.3, 90.0)
- added J1: USB_B_Micro, Connector_USB:USB_Micro-B_Molex_47346-0001, F.Cu at (220.9, 90.0)
- added J1: USB_B_Micro, Connector_USB:USB_Micro-B_Molex_47346-0001, F.Cu at (170.1, 90.0)
- added J1: USB_B_Micro, Connector_USB:USB_Micro-B_Molex_47346-0001, F.Cu at (17.7, 90.0)
- added J1: USB_B_Micro, Connector_USB:USB_Micro-B_Molex_47346-0001, F.Cu at (68.5, 90.0)
- added J1: USB_B_Micro, Connector_USB:USB_Micro-B_Molex_47346-0001, F.Cu at (119.3, 59.6)
- added J1: USB_B_Micro, Connector_USB:USB_Micro-B_Molex_47346-0001, F.Cu at (170.1, 59.6)
- added J1: USB_B_Micro, Connector_USB:USB_Micro-B_Molex_47346-0001, F.Cu at (220.9, 59.6)
- added J1: USB_B_Micro, Connector_USB:USB_Micro-B_Molex_47346-0001, F.Cu at (17.7, 59.6)
- added J1: USB_B_Micro, Connector_USB:USB_Micro-B_Molex_47346-0001, F.Cu at (17.7, 151.0)
- added J1: USB_B_Micro, Connector_USB:USB_Micro-B_Molex_47346-0001, F.Cu at (68.5, 59.6)
- added J1: USB_B_Micro, Connector_USB:USB_Micro-B_Molex_47346-0001, F.Cu at (220.9, 29.1)
- added J1: USB_B_Micro, Connector_USB:USB_Micro-B_Molex_47346-0001, F.Cu at (170.1, 29.1)
- added J1: USB_B_Micro, Connector_USB:USB_Micro-B_Molex_47346-0001, F.Cu at (119.3, 29.1)
- added J1: USB_B_Micro, Connector_USB:USB_Micro-B_Molex_47346-0001, F.Cu at (68.5, 29.1)
- added J1: USB_B_Micro, Connector_USB:USB_Micro-B_Molex_47346-0001, F.Cu at (220.9, 151.0)
- added J1: USB_B_Micro, Connector_USB:USB_Micro-B_Molex_47346-0001, F.Cu at (170.1, 151.0)
- added J1: USB_B_Micro, Connector_USB:USB_Micro-B_Molex_47346-0001, F.Cu at (68.5, 151.0)
- added J1: USB_B_Micro, Connector_USB:USB_Micro-B_Molex_47346-0001, F.Cu at (119.3, 120.5)
- added J1: USB_B_Micro, Connector_USB:USB_Micro-B_Molex_47346-0001, F.Cu at (170.1, 120.5)
- added J1: USB_B_Micro, Connector_USB:USB_Micro-B_Molex_47346-0001, F.Cu at (17.7, 120.5)
- added J1: USB_B_Micro, Connector_USB:USB_Micro-B_Molex_47346-0001, F.Cu at (220.9, 120.5)
- added J2: AVR-ISP-6, Connector_PinHeader_2.54mm:PinHeader_2x03_P2.54mm_Vertical_SMD, F.Cu at (154.5, 143.1)
- added J2: AVR-ISP-6, Connector_PinHeader_2.54mm:PinHeader_2x03_P2.54mm_Vertical_SMD, F.Cu at (205.3, 112.6)
- added J2: AVR-ISP-6, Connector_PinHeader_2.54mm:PinHeader_2x03_P2.54mm_Vertical_SMD, F.Cu at (154.5, 82.1)
- added J2: AVR-ISP-6, Connector_PinHeader_2.54mm:PinHeader_2x03_P2.54mm_Vertical_SMD, F.Cu at (205.3, 82.1)
- added J2: AVR-ISP-6, Connector_PinHeader_2.54mm:PinHeader_2x03_P2.54mm_Vertical_SMD, F.Cu at (256.1, 82.1)
- added J2: AVR-ISP-6, Connector_PinHeader_2.54mm:PinHeader_2x03_P2.54mm_Vertical_SMD, F.Cu at (52.9, 82.1)
- added J2: AVR-ISP-6, Connector_PinHeader_2.54mm:PinHeader_2x03_P2.54mm_Vertical_SMD, F.Cu at (103.7, 82.1)
- added J2: AVR-ISP-6, Connector_PinHeader_2.54mm:PinHeader_2x03_P2.54mm_Vertical_SMD, F.Cu at (154.5, 51.7)
- added J2: AVR-ISP-6, Connector_PinHeader_2.54mm:PinHeader_2x03_P2.54mm_Vertical_SMD, F.Cu at (205.3, 51.7)
- added J2: AVR-ISP-6, Connector_PinHeader_2.54mm:PinHeader_2x03_P2.54mm_Vertical_SMD, F.Cu at (256.1, 51.7)
- added J2: AVR-ISP-6, Connector_PinHeader_2.54mm:PinHeader_2x03_P2.54mm_Vertical_SMD, F.Cu at (52.9, 51.7)
- added J2: AVR-ISP-6, Connector_PinHeader_2.54mm:PinHeader_2x03_P2.54mm_Vertical_SMD, F.Cu at (256.1, 143.1)
- added J2: AVR-ISP-6, Connector_PinHeader_2.54mm:PinHeader_2x03_P2.54mm_Vertical_SMD, F.Cu at (103.7, 51.7)
- added J2: AVR-ISP-6, Connector_PinHeader_2.54mm:PinHeader_2x03_P2.54mm_Vertical_SMD, F.Cu at (256.1, 21.2)
- added J2: AVR-ISP-6, Connector_PinHeader_2.54mm:PinHeader_2x03_P2.54mm_Vertical_SMD, F.Cu at (205.3, 21.2)
- added J2: AVR-ISP-6, Connector_PinHeader_2.54mm:PinHeader_2x03_P2.54mm_Vertical_SMD, F.Cu at (154.5, 21.2)
- added J2: AVR-ISP-6, Connector_PinHeader_2.54mm:PinHeader_2x03_P2.54mm_Vertical_SMD, F.Cu at (103.7, 21.2)
- added J2: AVR-ISP-6, Connector_PinHeader_2.54mm:PinHeader_2x03_P2.54mm_Vertical_SMD, F.Cu at (52.9, 143.1)
- added J2: AVR-ISP-6, Connector_PinHeader_2.54mm:PinHeader_2x03_P2.54mm_Vertical_SMD, F.Cu at (205.3, 143.1)
- added J2: AVR-ISP-6, Connector_PinHeader_2.54mm:PinHeader_2x03_P2.54mm_Vertical_SMD, F.Cu at (103.7, 143.1)
- added J2: AVR-ISP-6, Connector_PinHeader_2.54mm:PinHeader_2x03_P2.54mm_Vertical_SMD, F.Cu at (154.5, 112.6)
- added J2: AVR-ISP-6, Connector_PinHeader_2.54mm:PinHeader_2x03_P2.54mm_Vertical_SMD, F.Cu at (103.7, 112.6)
- added J2: AVR-ISP-6, Connector_PinHeader_2.54mm:PinHeader_2x03_P2.54mm_Vertical_SMD, F.Cu at (256.1, 112.6)
- added J2: AVR-ISP-6, Connector_PinHeader_2.54mm:PinHeader_2x03_P2.54mm_Vertical_SMD, F.Cu at (52.9, 112.6)
- added JP1: Rest_connect, Jumper:SolderJumper-2_P1.3mm_Open_RoundedPad1.0x1.5mm, F.Cu at (196.5, 151.0)
- added JP1: Rest_connect, Jumper:SolderJumper-2_P1.3mm_Open_RoundedPad1.0x1.5mm, F.Cu at (94.9, 120.5)
- added JP1: Rest_connect, Jumper:SolderJumper-2_P1.3mm_Open_RoundedPad1.0x1.5mm, F.Cu at (196.5, 90.0)
- added JP1: Rest_connect, Jumper:SolderJumper-2_P1.3mm_Open_RoundedPad1.0x1.5mm, F.Cu at (145.7, 90.0)
- added JP1: Rest_connect, Jumper:SolderJumper-2_P1.3mm_Open_RoundedPad1.0x1.5mm, F.Cu at (247.3, 90.0)
- added JP1: Rest_connect, Jumper:SolderJumper-2_P1.3mm_Open_RoundedPad1.0x1.5mm, F.Cu at (44.1, 90.0)
- added JP1: Rest_connect, Jumper:SolderJumper-2_P1.3mm_Open_RoundedPad1.0x1.5mm, F.Cu at (94.9, 90.0)
- added JP1: Rest_connect, Jumper:SolderJumper-2_P1.3mm_Open_RoundedPad1.0x1.5mm, F.Cu at (145.7, 59.6)
- added JP1: Rest_connect, Jumper:SolderJumper-2_P1.3mm_Open_RoundedPad1.0x1.5mm, F.Cu at (196.5, 59.6)
- added JP1: Rest_connect, Jumper:SolderJumper-2_P1.3mm_Open_RoundedPad1.0x1.5mm, F.Cu at (247.3, 59.6)
- added JP1: Rest_connect, Jumper:SolderJumper-2_P1.3mm_Open_RoundedPad1.0x1.5mm, F.Cu at (44.1, 59.6)
- added JP1: Rest_connect, Jumper:SolderJumper-2_P1.3mm_Open_RoundedPad1.0x1.5mm, F.Cu at (145.7, 151.0)
- added JP1: Rest_connect, Jumper:SolderJumper-2_P1.3mm_Open_RoundedPad1.0x1.5mm, F.Cu at (94.9, 59.6)
- added JP1: Rest_connect, Jumper:SolderJumper-2_P1.3mm_Open_RoundedPad1.0x1.5mm, F.Cu at (247.3, 29.1)
- added JP1: Rest_connect, Jumper:SolderJumper-2_P1.3mm_Open_RoundedPad1.0x1.5mm, F.Cu at (196.5, 29.1)
- added JP1: Rest_connect, Jumper:SolderJumper-2_P1.3mm_Open_RoundedPad1.0x1.5mm, F.Cu at (145.7, 29.1)
- added JP1: Rest_connect, Jumper:SolderJumper-2_P1.3mm_Open_RoundedPad1.0x1.5mm, F.Cu at (94.9, 29.1)
- added JP1: Rest_connect, Jumper:SolderJumper-2_P1.3mm_Open_RoundedPad1.0x1.5mm, F.Cu at (44.1, 151.0)
- added JP1: Rest_connect, Jumper:SolderJumper-2_P1.3mm_Open_RoundedPad1.0x1.5mm, F.Cu at (247.3, 151.0)
- added JP1: Rest_connect, Jumper:SolderJumper-2_P1.3mm_Open_RoundedPad1.0x1.5mm, F.Cu at (94.9, 151.0)
- added JP1: Rest_connect, Jumper:SolderJumper-2_P1.3mm_Open_RoundedPad1.0x1.5mm, F.Cu at (196.5, 120.5)
- added JP1: Rest_connect, Jumper:SolderJumper-2_P1.3mm_Open_RoundedPad1.0x1.5mm, F.Cu at (145.7, 120.5)
- added JP1: Rest_connect, Jumper:SolderJumper-2_P1.3mm_Open_RoundedPad1.0x1.5mm, F.Cu at (44.1, 120.5)
- added JP1: Rest_connect, Jumper:SolderJumper-2_P1.3mm_Open_RoundedPad1.0x1.5mm, F.Cu at (247.3, 120.5)
- added JP2: USB_power, Jumper:SolderJumper-2_P1.3mm_Bridged2Bar_RoundedPad1.0x1.5mm, F.Cu at (157.6, 163.3)
- added JP2: USB_power, Jumper:SolderJumper-2_P1.3mm_Bridged2Bar_RoundedPad1.0x1.5mm, F.Cu at (56.0, 132.8)
- added JP2: USB_power, Jumper:SolderJumper-2_P1.3mm_Bridged2Bar_RoundedPad1.0x1.5mm, F.Cu at (157.6, 102.3)
- added JP2: USB_power, Jumper:SolderJumper-2_P1.3mm_Bridged2Bar_RoundedPad1.0x1.5mm, F.Cu at (208.4, 102.3)
- added JP2: USB_power, Jumper:SolderJumper-2_P1.3mm_Bridged2Bar_RoundedPad1.0x1.5mm, F.Cu at (259.2, 102.3)
- added JP2: USB_power, Jumper:SolderJumper-2_P1.3mm_Bridged2Bar_RoundedPad1.0x1.5mm, F.Cu at (106.8, 102.3)
- added JP2: USB_power, Jumper:SolderJumper-2_P1.3mm_Bridged2Bar_RoundedPad1.0x1.5mm, F.Cu at (56.0, 102.3)
- added JP2: USB_power, Jumper:SolderJumper-2_P1.3mm_Bridged2Bar_RoundedPad1.0x1.5mm, F.Cu at (157.6, 71.8)
- added JP2: USB_power, Jumper:SolderJumper-2_P1.3mm_Bridged2Bar_RoundedPad1.0x1.5mm, F.Cu at (208.4, 71.8)
- added JP2: USB_power, Jumper:SolderJumper-2_P1.3mm_Bridged2Bar_RoundedPad1.0x1.5mm, F.Cu at (259.2, 71.8)
- added JP2: USB_power, Jumper:SolderJumper-2_P1.3mm_Bridged2Bar_RoundedPad1.0x1.5mm, F.Cu at (56.0, 71.8)
- added JP2: USB_power, Jumper:SolderJumper-2_P1.3mm_Bridged2Bar_RoundedPad1.0x1.5mm, F.Cu at (208.4, 163.3)
- added JP2: USB_power, Jumper:SolderJumper-2_P1.3mm_Bridged2Bar_RoundedPad1.0x1.5mm, F.Cu at (106.8, 71.8)
- added JP2: USB_power, Jumper:SolderJumper-2_P1.3mm_Bridged2Bar_RoundedPad1.0x1.5mm, F.Cu at (259.2, 41.3)
- added JP2: USB_power, Jumper:SolderJumper-2_P1.3mm_Bridged2Bar_RoundedPad1.0x1.5mm, F.Cu at (208.4, 41.3)
- added JP2: USB_power, Jumper:SolderJumper-2_P1.3mm_Bridged2Bar_RoundedPad1.0x1.5mm, F.Cu at (157.6, 41.3)
- added JP2: USB_power, Jumper:SolderJumper-2_P1.3mm_Bridged2Bar_RoundedPad1.0x1.5mm, F.Cu at (106.8, 41.3)
- added JP2: USB_power, Jumper:SolderJumper-2_P1.3mm_Bridged2Bar_RoundedPad1.0x1.5mm, F.Cu at (106.8, 163.3)
- added JP2: USB_power, Jumper:SolderJumper-2_P1.3mm_Bridged2Bar_RoundedPad1.0x1.5mm, F.Cu at (259.2, 163.3)
- added JP2: USB_power, Jumper:SolderJumper-2_P1.3mm_Bridged2Bar_RoundedPad1.0x1.5mm, F.Cu at (56.0, 163.3)
- added JP2: USB_power, Jumper:SolderJumper-2_P1.3mm_Bridged2Bar_RoundedPad1.0x1.5mm, F.Cu at (157.6, 132.8)
- added JP2: USB_power, Jumper:SolderJumper-2_P1.3mm_Bridged2Bar_RoundedPad1.0x1.5mm, F.Cu at (259.2, 132.8)
- added JP2: USB_power, Jumper:SolderJumper-2_P1.3mm_Bridged2Bar_RoundedPad1.0x1.5mm, F.Cu at (106.8, 132.8)
- added JP2: USB_power, Jumper:SolderJumper-2_P1.3mm_Bridged2Bar_RoundedPad1.0x1.5mm, F.Cu at (208.4, 132.8)
- added R1: 1k, Resistor_SMD:R_0805_2012Metric_Pad1.15x1.40mm_HandSolder, F.Cu at (132.6, 142.8)
- added R1: 1k, Resistor_SMD:R_0805_2012Metric_Pad1.15x1.40mm_HandSolder, F.Cu at (81.8, 112.4)
- added R1: 1k, Resistor_SMD:R_0805_2012Metric_Pad1.15x1.40mm_HandSolder, F.Cu at (132.6, 81.9)
- added R1: 1k, Resistor_SMD:R_0805_2012Metric_Pad1.15x1.40mm_HandSolder, F.Cu at (183.4, 81.9)
- added R1: 1k, Resistor_SMD:R_0805_2012Metric_Pad1.15x1.40mm_HandSolder, F.Cu at (234.2, 81.9)
- added R1: 1k, Resistor_SMD:R_0805_2012Metric_Pad1.15x1.40mm_HandSolder, F.Cu at (31.0, 81.9)
- added R1: 1k, Resistor_SMD:R_0805_2012Metric_Pad1.15x1.40mm_HandSolder, F.Cu at (81.8, 81.9)
- added R1: 1k, Resistor_SMD:R_0805_2012Metric_Pad1.15x1.40mm_HandSolder, F.Cu at (132.6, 51.4)
- added R1: 1k, Resistor_SMD:R_0805_2012Metric_Pad1.15x1.40mm_HandSolder, F.Cu at (183.4, 51.4)
- added R1: 1k, Resistor_SMD:R_0805_2012Metric_Pad1.15x1.40mm_HandSolder, F.Cu at (234.2, 51.4)
- added R1: 1k, Resistor_SMD:R_0805_2012Metric_Pad1.15x1.40mm_HandSolder, F.Cu at (31.0, 51.4)
- added R1: 1k, Resistor_SMD:R_0805_2012Metric_Pad1.15x1.40mm_HandSolder, F.Cu at (183.4, 142.8)
- added R1: 1k, Resistor_SMD:R_0805_2012Metric_Pad1.15x1.40mm_HandSolder, F.Cu at (81.8, 51.4)
- added R1: 1k, Resistor_SMD:R_0805_2012Metric_Pad1.15x1.40mm_HandSolder, F.Cu at (234.2, 20.9)
- added R1: 1k, Resistor_SMD:R_0805_2012Metric_Pad1.15x1.40mm_HandSolder, F.Cu at (183.4, 20.9)
- added R1: 1k, Resistor_SMD:R_0805_2012Metric_Pad1.15x1.40mm_HandSolder, F.Cu at (132.6, 20.9)
- added R1: 1k, Resistor_SMD:R_0805_2012Metric_Pad1.15x1.40mm_HandSolder, F.Cu at (81.8, 20.9)
- added R1: 1k, Resistor_SMD:R_0805_2012Metric_Pad1.15x1.40mm_HandSolder, F.Cu at (234.2, 142.8)
- added R1: 1k, Resistor_SMD:R_0805_2012Metric_Pad1.15x1.40mm_HandSolder, F.Cu at (31.0, 142.8)
- added R1: 1k, Resistor_SMD:R_0805_2012Metric_Pad1.15x1.40mm_HandSolder, F.Cu at (81.8, 142.8)
- added R1: 1k, Resistor_SMD:R_0805_2012Metric_Pad1.15x1.40mm_HandSolder, F.Cu at (132.6, 112.4)
- added R1: 1k, Resistor_SMD:R_0805_2012Metric_Pad1.15x1.40mm_HandSolder, F.Cu at (183.4, 112.4)
- added R1: 1k, Resistor_SMD:R_0805_2012Metric_Pad1.15x1.40mm_HandSolder, F.Cu at (234.2, 112.4)
- added R1: 1k, Resistor_SMD:R_0805_2012Metric_Pad1.15x1.40mm_HandSolder, F.Cu at (31.0, 112.4)
- added R4: 0, Resistor_SMD:R_0805_2012Metric_Pad1.15x1.40mm_HandSolder, F.Cu at (202.6, 149.4)
- added R4: 0, Resistor_SMD:R_0805_2012Metric_Pad1.15x1.40mm_HandSolder, F.Cu at (101.0, 118.9)
- added R4: 0, Resistor_SMD:R_0805_2012Metric_Pad1.15x1.40mm_HandSolder, F.Cu at (202.6, 88.4)
- added R4: 0, Resistor_SMD:R_0805_2012Metric_Pad1.15x1.40mm_HandSolder, F.Cu at (151.8, 88.4)
- added R4: 0, Resistor_SMD:R_0805_2012Metric_Pad1.15x1.40mm_HandSolder, F.Cu at (253.4, 88.4)
- added R4: 0, Resistor_SMD:R_0805_2012Metric_Pad1.15x1.40mm_HandSolder, F.Cu at (50.2, 88.4)
- added R4: 0, Resistor_SMD:R_0805_2012Metric_Pad1.15x1.40mm_HandSolder, F.Cu at (101.0, 88.4)
- added R4: 0, Resistor_SMD:R_0805_2012Metric_Pad1.15x1.40mm_HandSolder, F.Cu at (151.8, 57.9)
- added R4: 0, Resistor_SMD:R_0805_2012Metric_Pad1.15x1.40mm_HandSolder, F.Cu at (202.6, 57.9)
- added R4: 0, Resistor_SMD:R_0805_2012Metric_Pad1.15x1.40mm_HandSolder, F.Cu at (253.4, 57.9)
- added R4: 0, Resistor_SMD:R_0805_2012Metric_Pad1.15x1.40mm_HandSolder, F.Cu at (50.2, 57.9)
- added R4: 0, Resistor_SMD:R_0805_2012Metric_Pad1.15x1.40mm_HandSolder, F.Cu at (253.4, 149.4)
- added R4: 0, Resistor_SMD:R_0805_2012Metric_Pad1.15x1.40mm_HandSolder, F.Cu at (101.0, 57.9)
- added R4: 0, Resistor_SMD:R_0805_2012Metric_Pad1.15x1.40mm_HandSolder, F.Cu at (253.4, 27.4)
- added R4: 0, Resistor_SMD:R_0805_2012Metric_Pad1.15x1.40mm_HandSolder, F.Cu at (202.6, 27.4)
- added R4: 0, Resistor_SMD:R_0805_2012Metric_Pad1.15x1.40mm_HandSolder, F.Cu at (151.8, 27.4)
- added R4: 0, Resistor_SMD:R_0805_2012Metric_Pad1.15x1.40mm_HandSolder, F.Cu at (101.0, 27.4)
- added R4: 0, Resistor_SMD:R_0805_2012Metric_Pad1.15x1.40mm_HandSolder, F.Cu at (151.8, 149.4)
- added R4: 0, Resistor_SMD:R_0805_2012Metric_Pad1.15x1.40mm_HandSolder, F.Cu at (50.2, 149.4)
- added R4: 0, Resistor_SMD:R_0805_2012Metric_Pad1.15x1.40mm_HandSolder, F.Cu at (101.0, 149.4)
- added R4: 0, Resistor_SMD:R_0805_2012Metric_Pad1.15x1.40mm_HandSolder, F.Cu at (202.6, 118.9)
- added R4: 0, Resistor_SMD:R_0805_2012Metric_Pad1.15x1.40mm_HandSolder, F.Cu at (253.4, 118.9)
- added R4: 0, Resistor_SMD:R_0805_2012Metric_Pad1.15x1.40mm_HandSolder, F.Cu at (151.8, 118.9)
- added R4: 0, Resistor_SMD:R_0805_2012Metric_Pad1.15x1.40mm_HandSolder, F.Cu at (50.2, 118.9)
- added R5: 10k, Resistor_SMD:R_0805_2012Metric_Pad1.15x1.40mm_HandSolder, F.Cu at (156.8, 152.6)
- added R5: 10k, Resistor_SMD:R_0805_2012Metric_Pad1.15x1.40mm_HandSolder, F.Cu at (106.0, 122.1)
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Routing:
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Other:
- board size 44.8 x 29 mm -> 248 x 150.9 mm
- net class Default: clearance 0.25 -> 0.2
- rule trace_clearance: 0.25 -> 0.2

Commit message: update
Parts:
- removed the G*** at (18.4, 41.9)
